File: lincal.kicad_pcb (KiCad board)
At the start: 4 copper layers, 250 x 150 mm, 657 parts, among them J61 Conn_01x01_Socket, J62 Conn_01x01_Socket, J71 Conn_01x01_Socket, J72 Conn_01x01_Socket, J73 Conn_01x01_Socket, J74 Conn_01x01_Socket, J75 Conn_01x01_Socket, J76 Conn_01x01_Socket, J81 Conn_01x03_Pin, J82 Conn_Coaxial, J83 Conn_Coaxial, J84 Conn_01x02_Pin, J85 USB_C_Receptacle_USB2.0_16P, J86 Conn_01x02_Pin, K21 G6K-2FY, 5V, K22 G6K-2FY, 5V, Q201 AO3400A, Q202 AO3401A, Q203 AO3400A, Q204 AO3400A, Q205 AO3400A, Q206 AO3400A, Q207 AO3400A, Q251 AO3400A, Q252 AO3401A, Q253 AO3400A, Q254 AO3400A, Q255 AO3400A, Q256 AO3400A, Q257 AO3400A, Q81 Si2301CDS, Q82 AO3400A, SW81 SW_Push, SW82 SW_Push, U11 OPA2189DGK, U12 TMUX1108PW, U18 DG419D, U19 TCA0372, U21 OPA828DGN, U22 OPA2197D, U23 DG419D, U25 OPA828DGN, U26 OPA2197D, U27 DG419D, U30 LTC2752B, U301 OPA2197D, U302 OPA2197D, U303 OPA2197D, U304 OPA2197D, U305 DG419D, U31 OPA2189DGK, U32 OPA2388DGK, U321 DG419D, U33 OPA2388DGK, U341 DG419D, U35 LTC2752B, U36 OPA2189DGK, U361 DG419D, U37 OPA2388DGK, U38 OPA2388DGK, U41 TPS7A8801RTJR, U42 TPS7A8801RTJR, U43 TPS61252DSG, U44 TPSM863252RDXR, U45 TPS7A3301RGW, U46 TPSM863252RDXR, U51 ADP5071ACPZ, U52 TPS7A4700xRGW, U53 TPS7A3301RGW, U6 REF7050, U61 OPA2189DGK, U7 AD7177-2BRUZ, U70 TG2520SMN-16M-MCG, U704 OPA2197D, U706 OPA2197D, U707 OPA2197D, U71 TMUX6104, U72 TMUX6104, U73 OPA2388DGK, U74 THS4521IDGK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

Commit message: Whew.  DACs routed
Parts:
- removed the R441 at (107.7, 83.7)
- removed TP49: TestPoint, Parts:TestPoint
- added C102: 1u, Capacitor_SMD:C_0402_1005Metric, F.Cu at (256.5, 192.5)
- added C462: 1u, Capacitor_SMD:C_0402_1005Metric, F.Cu at (132.2, 168.8)
- added C67: 10u, Capacitor_SMD:C_0603_1608Metric, F.Cu at (118.6, 63.2)
- added C68: 1u, Capacitor_SMD:C_0402_1005Metric, F.Cu at (122.0, 62.9)
- added C741: 10u, Capacitor_SMD:C_0603_1608Metric, F.Cu at (211.0, 90.3)
- added C742: 0n1, Capacitor_SMD:C_0402_1005Metric, F.Cu at (195.3, 67.2)
- added C743: 0n1, Capacitor_SMD:C_0402_1005Metric, F.Cu at (195.3, 69.1)
- added C744: 0n1, Capacitor_SMD:C_0402_1005Metric, F.Cu at (195.3, 71.0)
- added C745: 0n1, Capacitor_SMD:C_0402_1005Metric, F.Cu at (195.3, 73.0)
- added L63: 100, Inductor_SMD:L_0603_1608Metric, F.Cu at (118.6, 65.7)
- added R118: 100, Resistor_SMD:R_0402_1005Metric, F.Cu at (254.0, 193.3)
- added R732: 1, Resistor_SMD:R_0603_1608Metric, F.Cu at (211.0, 92.8)
- added R753: 10k, Resistor_SMD:R_0402_1005Metric, F.Cu at (214.5, 90.0)
- C201, C251: footprint Capacitor_THT:C_Rect_L31.5mm_W15.0mm_P27.50mm_MKS4 -> Parts:C_Rect_L31.5mm_W15.0mm_P27.50mm_MKS4
- C202, C252: value 0n1 -> 1n; footprint Capacitor_SMD:C_0603_1608Metric -> Capacitor_SMD:C_0402_1005Metric
- C204, C254: value 100p -> 0n1
- C205, C255, C313, C326, C352, C372: value 10n -> 0n1; footprint Capacitor_SMD:C_0603_1608Metric -> Capacitor_SMD:C_0402_1005Metric
- NT31, NT32, NT33, NT34: footprint NetTie:NetTie-2_SMD_Pad0.5mm -> Parts:NetTie-2_SMD_Pad0.5mm; moved to B.Cu
- Q201, Q202, Q203, Q204, Q205, Q206, Q207, Q251, Q252, Q253, Q254, Q255, Q256, Q257, Q81, Q82: footprint Package_TO_SOT_SMD:SOT-23 -> Parts:SOT-23
- R211, R261: value 100 -> 330
- R67: footprint Resistor_SMD:R_0402_1005Metric -> Resistor_SMD:R_0603_1608Metric
- R754: renamed from R732; value 1 -> 10k; footprint Resistor_SMD:R_0603_1608Metric -> Resistor_SMD:R_0402_1005Metric
- U11, U31, U36, U61, U75, U76, U78: footprint Package_SO:MSOP-8_3x3mm_P0.65mm -> Parts:OPA2189
- U21, U25: footprint Package_SO:HVSSOP-8-1EP_3x3mm_P0.65mm_EP1.57x1.89mm -> Parts:VSSOP-8-1EP_3x3mm_P0.65mm_EP1.57x1.89mm
- U22, U26, U301, U704, U706, U707: footprint Package_SO:SOIC-8_3.9x4.9mm_P1.27mm -> Parts:OPA2197
- U30, U35: footprint Package_QFP:LQFP-48_7x7mm_P0.5mm -> Parts:LQFP-48_7x7mm_P0.5mm
- U32, U33, U37, U38, U73, U77: footprint Package_SO:MSOP-8_3x3mm_P0.65mm -> Parts:OPA2388
- U321: renamed from U302; footprint Package_SO:SOIC-8_3.9x4.9mm_P1.27mm -> Parts:OPA2197
- U341: renamed from U303; footprint Package_SO:SOIC-8_3.9x4.9mm_P1.27mm -> Parts:OPA2197
- U361: renamed from U304; footprint Package_SO:SOIC-8_3.9x4.9mm_P1.27mm -> Parts:OPA2197
- U74: footprint Package_SO:VSSOP-8_3x3mm_P0.65mm -> Parts:MSOP-8_3x3mm_P0.65mm
- moved C313 157.0 mm to (291.5, 194.2), turned to -90 degrees
- moved C311 150.0 mm to (291.3, 196.6), turned to -90 degrees
- moved C385 147.8 mm to (296.4, 191.4)
- moved C325 147.2 mm to (298.7, 197.4), turned to -90 degrees
- moved C301 146.2 mm to (282.3, 184.7)
- moved C312 145.7 mm to (314.7, 186.2), turned to -90 degrees
- moved U31 145.0 mm to (295.0, 194.9)
- moved C382 144.8 mm to (295.8, 192.6), turned to 180 degrees
- moved C381 144.1 mm to (294.0, 191.1)
- moved R301 143.9 mm to (284.6, 185.5), turned to -90 degrees
- moved L31 142.7 mm to (293.4, 192.3)
- moved C326 142.4 mm to (298.5, 194.9), turned to -90 degrees
- moved C302 141.6 mm to (274.0, 186.2), turned to -90 degrees
- moved R302 141.2 mm to (282.3, 186.2)
- moved R315 141.0 mm to (290.1, 196.6), turned to -90 degrees
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- renumbered C462 to C463, C463 to C464, C464 to C465, C465 to C466, C466 to C467, C68 to C66, C67 to C69, R118 to R114, R120 to R115, R119 to R116, R121 to R117, R116 to R120, R117 to R121, R442 to R441, R443 to R442, R444 to R443, U305 to U302, U321 to U322, U341 to U342, U361 to U362
Connections:
- net Net-(C203-Pad2) renamed /Sample Hold 1/Drive
- net Net-(C253-Pad2) renamed /Sample Hold 2/Drive
- net Net-(C302-Pad1) renamed /DAC2752-1A/FREF
- net Net-(C313-Pad1) renamed /DAC2752-1A/RIN
- net Net-(C342-Pad1) renamed /DAC2752-2A/FREF
- net Net-(C352-Pad1) renamed /DAC2752-2A/RIN
- net Net-(D51-A) renamed /18V/Sp
- net Net-(D52-K) renamed /18V/Sn
- net Net-(R307-Pad1) renamed /DAC2752-1A/ROFS
- net Net-(R327-Pad1) renamed /DAC2752-1B/ROFS
- net Net-(R347-Pad1) renamed /DAC2752-2A/ROFS
- net Net-(R367-Pad1) renamed /DAC2752-2B/ROFS
- net Net-(U21-+) renamed /Sample Hold 1/SH
- net Net-(U25-+) renamed /Sample Hold 2/SH
- net Net-(U30A-RCOMA) renamed /DAC2752-1A/RCOM
- net Net-(U31A--) renamed /DAC2752-1A/RSense
- net Net-(U35A-RCOMA) renamed /DAC2752-2A/RCOM
- net Net-(U36A--) renamed /DAC2752-2A/RSense
- net Net-(U41A-EN1) renamed /Low Voltage Power/I5VA
- net Net-(U41B-EN2) renamed /Low Voltage Power/I5V6A
- net Net-(U42A-EN1) renamed /Low Voltage Power/I3V3A
- net Net-(U42B-EN2) renamed /Low Voltage Power/I2V5
- net Net-(U44-EN) renamed /Low Voltage Power/I3V3
- net Net-(U46-VIN) renamed /Low Voltage Power/Im3V3
- net Net-(U51-FB1) renamed /18V/FB1
- net Net-(U51-FB2) renamed /18V/FB2
- net Net-(U51-VREF) renamed /18V/VRef
- C104 pad 2: GND -> GNDPWR
- C202 pad 2: Net-(U19A-+) -> Net-(U19B-+)
- C252 pad 2: Net-(U19B-+) -> Net-(U19A-+)
- C303 pad 1: Net-(C303-Pad1) -> /DAC2752-1A/IOUT1
- C303 pad 2: Net-(U30A-IOUT1A) -> /DAC2752-1A/Force
- C306 pad 1: Net-(C306-Pad1) -> /DAC2752-1A/Force
- C312 pad 1: Net-(C312-Pad1) -> /DAC2752-1B/FREF
- C326 pad 1: Net-(C326-Pad1) -> /DAC2752-1B/RIN
- C326 pad 2: Net-(U31B--) -> /DAC2752-1B/RSense
- C328 pad 1: Net-(C328-Pad1) -> /DAC2752-1B/IOUT1
- C328 pad 2: Net-(U30B-IOUT1B) -> /DAC2752-1B/Force
- C329 pad 1: Net-(C329-Pad1) -> /DAC2752-1B/Force
- C330 pad 2: Net-(U33B--) -> Net-(U33A--)
- C331 pad 2: Net-(U33A--) -> Net-(U33B--)
- C343 pad 1: Net-(C343-Pad1) -> /DAC2752-2A/IOUT1
- C343 pad 2: Net-(U35A-IOUT1A) -> /DAC2752-2A/Force
- C345 pad 1: Net-(C345-Pad1) -> /DAC2752-2A/Force
- C361 pad 2: Net-(U38A--) -> Net-(U38B--)
- C362 pad 1: Net-(C362-Pad1) -> /DAC2752-2B/FREF
- C363 pad 1: Net-(C363-Pad1) -> /DAC2752-2B/IOUT1
- C363 pad 2: Net-(U35B-IOUT1B) -> /DAC2752-2B/Force
- C364 pad 2: Net-(U38B--) -> Net-(U38A--)
- C366 pad 1: Net-(C366-Pad1) -> /DAC2752-2B/Force
- C372 pad 1: Net-(C372-Pad1) -> /DAC2752-2B/RIN
- C372 pad 2: Net-(U36B--) -> /DAC2752-2B/RSense
- C441 pad 1: Net-(U43-EN) -> /Low Voltage Power/I6V
- C442 pad 1: Net-(U43-EN) -> /Low Voltage Power/I6V
- J61 pad 1: Ref5V -> Net-(J61-Pin_1)
- L441 pad 1: Net-(U43-EN) -> /Low Voltage Power/I6V
- L45 pad 2: Net-(U43-EN) -> /Low Voltage Power/I6V
- NT31 pad 2: Net-(U30A-IOUT2AF) -> /DAC2752-1A/IOUT2
- NT32 pad 2: Net-(U30B-IOUT2BF) -> /DAC2752-1B/IOUT2
- NT33 pad 2: Net-(U35A-IOUT2AF) -> /DAC2752-2A/IOUT2
- NT34 pad 2: Net-(U35B-IOUT2BF) -> /DAC2752-2B/IOUT2
- R108 pad 1: /Offset Voltage Ladder/5V -> /Offset Voltage Ladder/L5V
- R202 pad 1: Net-(U19A--) -> Net-(U19B--)
- R203 pad 1: Net-(U19A--) -> Net-(U19B--)
- R204 pad 1: Net-(U19A--) -> Net-(U19B--)
- R205 pad 1: Net-(U19A--) -> Net-(U19B--)
- R206 pad 1: Net-(U19A--) -> Net-(U19B--)
- R252 pad 1: Net-(U19B--) -> Net-(U19A--)
- R253 pad 1: Net-(U19B--) -> Net-(U19A--)
- R254 pad 1: Net-(U19B--) -> Net-(U19A--)
- R255 pad 1: Net-(U19B--) -> Net-(U19A--)
- R256 pad 1: Net-(U19B--) -> Net-(U19A--)
- R305 pad 2: Net-(U30A-IOUT2AF) -> Net-(U30A-IOUT2AS)
- R306 pad 1: Net-(U30A-IOUT2AF) -> Net-(U30A-IOUT2AS)
- R309 pad 2: Net-(U30A-IOUT2AF) -> GND
- R313 pad 1: Net-(C306-Pad1) -> /DAC2752-1A/Force
- R313 pad 2: Net-(C303-Pad1) -> /DAC2752-1A/RFB
- R314 pad 1: Net-(C306-Pad1) -> /DAC2752-1A/Force
- R314 pad 2: Net-(C303-Pad1) -> /DAC2752-1A/RFB
- R321 pad 1: Net-(U33A--) -> Net-(U33B--)
- R322 pad 2: Net-(U33A--) -> Net-(U33B--)
- R323 pad 1: Net-(U302A--) -> Net-(U321B--)
- R324 pad 2: Net-(U302A--) -> Net-(U321B--)
- R325 pad 1: Net-(C312-Pad1) -> /DAC2752-1B/FREF
- R325 pad 2: Net-(U30B-IOUT2BF) -> Net-(U30B-IOUT2BS)
- R326 pad 1: Net-(U30B-IOUT2BF) -> Net-(U30B-IOUT2BS)
- R327 pad 2: Net-(C326-Pad1) -> /DAC2752-1B/RIN
- R328 pad 2: Net-(C326-Pad1) -> /DAC2752-1B/RIN
- R329 pad 1: Net-(U33B--) -> Net-(U33A--)
- R329 pad 2: Net-(U30B-IOUT2BF) -> GND
- R330 pad 2: Net-(U33B--) -> Net-(U33A--)
- R331 pad 1: Net-(U302B--) -> Net-(U321A--)
- R332 pad 2: Net-(U302B--) -> Net-(U321A--)
- R333 pad 1: Net-(C329-Pad1) -> /DAC2752-1B/Force
- R333 pad 2: Net-(C328-Pad1) -> /DAC2752-1B/RFB
- R334 pad 1: Net-(C329-Pad1) -> /DAC2752-1B/Force
- R334 pad 2: Net-(C328-Pad1) -> /DAC2752-1B/RFB
- R345 pad 2: Net-(U35A-IOUT2AF) -> Net-(U35A-IOUT2AS)
- R346 pad 1: Net-(U35A-IOUT2AF) -> Net-(U35A-IOUT2AS)
- R349 pad 2: Net-(U35A-IOUT2AF) -> GND
- R353 pad 1: Net-(C345-Pad1) -> /DAC2752-2A/Force
- R353 pad 2: Net-(C343-Pad1) -> /DAC2752-2A/RFB
- R354 pad 1: Net-(C345-Pad1) -> /DAC2752-2A/Force
- R354 pad 2: Net-(C343-Pad1) -> /DAC2752-2A/RFB
- R361 pad 1: Net-(U38A--) -> Net-(U38B--)
- R362 pad 2: Net-(U38A--) -> Net-(U38B--)
- R363 pad 1: Net-(U304A--) -> Net-(U361B--)
- R364 pad 2: Net-(U304A--) -> Net-(U361B--)
- R365 pad 1: Net-(C362-Pad1) -> /DAC2752-2B/FREF
- R365 pad 2: Net-(U35B-IOUT2BF) -> Net-(U35B-IOUT2BS)
- R366 pad 1: Net-(U35B-IOUT2BF) -> Net-(U35B-IOUT2BS)
- R367 pad 2: Net-(C372-Pad1) -> /DAC2752-2B/RIN
- R368 pad 2: Net-(C372-Pad1) -> /DAC2752-2B/RIN
- R369 pad 1: Net-(U38B--) -> Net-(U38A--)
- R369 pad 2: Net-(U35B-IOUT2BF) -> GND
- R370 pad 2: Net-(U38B--) -> Net-(U38A--)
- R371 pad 1: Net-(U304B--) -> Net-(U361A--)
- R372 pad 2: Net-(U304B--) -> Net-(U361A--)
- R373 pad 1: Net-(C366-Pad1) -> /DAC2752-2B/Force
- R373 pad 2: Net-(C363-Pad1) -> /DAC2752-2B/RFB
- R374 pad 1: Net-(C366-Pad1) -> /DAC2752-2B/Force
- R374 pad 2: Net-(C363-Pad1) -> /DAC2752-2B/RFB
- R722 pad 2: Net-(U74-V_{OCM}) -> Net-(C741-Pad1)
- R739 pad 1: Net-(U706A--) -> Net-(U706B--)
- R740 pad 1: Net-(U706B--) -> Net-(U706A--)
- R744 pad 1: Net-(R744-Pad1) -> Net-(C743-Pad2)
- R745 pad 1: Net-(R744-Pad1) -> Net-(C743-Pad2)
- R746 pad 1: Net-(R744-Pad1) -> Net-(U707A--)
- R746 pad 2: Net-(U707A--) -> Net-(C743-Pad2)
- R747 pad 1: Net-(U707A--) -> Net-(U707B--)
- R748 pad 1: Net-(U707B--) -> Net-(U707A--)
- R749 pad 1: Net-(R749-Pad1) -> Net-(U707B--)
- R749 pad 2: Net-(U707B--) -> Net-(C745-Pad2)
- R750 pad 1: Net-(R749-Pad1) -> Net-(C745-Pad2)
- R751 pad 1: Net-(R749-Pad1) -> Net-(C745-Pad2)
- R754 pad 1: Net-(C728-Pad1) -> Net-(C741-Pad1)
- R754 pad 2: /FDA/Out- -> +5VA
- TP303 pad 1: Net-(C303-Pad1) -> /DAC2752-1A/RFB
- TP304 pad 1: Net-(C306-Pad1) -> /DAC2752-1A/Force
- TP321 pad 1: Net-(C326-Pad1) -> /DAC2752-1B/RIN
- TP323 pad 1: Net-(C328-Pad1) -> /DAC2752-1B/RFB
- TP324 pad 1: Net-(C329-Pad1) -> /DAC2752-1B/Force
- TP343 pad 1: Net-(C343-Pad1) -> /DAC2752-2A/RFB
- TP344 pad 1: Net-(C345-Pad1) -> /DAC2752-2A/Force
- TP361 pad 1: Net-(C372-Pad1) -> /DAC2752-2B/RIN
- TP363 pad 1: Net-(C363-Pad1) -> /DAC2752-2B/RFB
- TP364 pad 1: Net-(C366-Pad1) -> /DAC2752-2B/Force
- TP51 pad 1: /18V/R18in -> +20V
- TP53 pad 1: /18V/RM18Vin -> -20V
- U11 pad 5: GNDPWR -> Net-(U11B-+)
- U11 pad 6: Net-(U11B--) -> /Offset Voltage Ladder/L5V
- U11 pad 7: Net-(U11B--) -> /Offset Voltage Ladder/L5V
- U21 pad 9: GND -> GNDPWR
- U22 pad 1: Net-(U19A-+) -> Net-(U19B-+)
- U25 pad 9: GND -> GNDPWR
- U26 pad 1: Net-(U19B-+) -> Net-(U19A-+)
- U30 pad 28: Net-(U30B-IOUT2BF) -> /DAC2752-1B/IOUT2
- U30 pad 29: Net-(U30B-IOUT2BF) -> Net-(U30B-IOUT2BS)
- U30 pad 31: Net-(C326-Pad1) -> /DAC2752-1B/RSense
- U30 pad 32: Net-(U31B--) -> /DAC2752-1B/RIN
- U30 pad 34: Net-(U30B-RCOMB) -> /DAC2752-1B/RCOM
- U30 pad 35: Net-(C312-Pad1) -> /DAC2752-1B/FREF
- U30 pad 36: Net-(C312-Pad1) -> /DAC2752-1B/FREF
- U30 pad 39: Net-(U321-S1) -> /DAC2752-1B/RFB
- U30 pad 40: Net-(C328-Pad1) -> /DAC2752-1B/Sense
- U30 pad 41: Net-(U30B-IOUT1B) -> /DAC2752-1B/IOUT1
- U30 pad 44: Net-(U30A-IOUT1A) -> /DAC2752-1A/IOUT1
- U30 pad 45: Net-(C303-Pad1) -> /DAC2752-1A/Sense
- U30 pad 46: Net-(U305-S1) -> /DAC2752-1A/RFB
- U30 pad 8: Net-(U30A-IOUT2AF) -> Net-(U30A-IOUT2AS)
- U30 pad 9: Net-(U30A-IOUT2AF) -> /DAC2752-1A/IOUT2
- U301 pad 7: Net-(C306-Pad1) -> /DAC2752-1A/Force
- U302 pad 2: Net-(U305-S1) -> /DAC2752-1A/Sense
- U31 pad 6: Net-(U31B--) -> /DAC2752-1B/RSense
- U31 pad 7: Net-(C326-Pad1) -> /DAC2752-1B/RIN
- U32 pad 5: Net-(U30A-IOUT1A) -> /DAC2752-1A/IOUT1
- U321 pad 1: Net-(C312-Pad1) -> /DAC2752-1B/Force
- U321 pad 2: Net-(U302A--) -> Net-(U321A--)
- U321 pad 6: Net-(U302B--) -> Net-(U321B--)
- U321 pad 7: Net-(C329-Pad1) -> /DAC2752-1B/FREF
- U322 pad 2: Net-(U321-S1) -> /DAC2752-1B/Sense
- U33 pad 1: Net-(C331-Pad1) -> Net-(C330-Pad1)
- U33 pad 3: Net-(U30B-RCOMB) -> /DAC2752-1B/IOUT1
- U33 pad 5: Net-(U30B-IOUT1B) -> /DAC2752-1B/RCOM
- U33 pad 7: Net-(C330-Pad1) -> Net-(C331-Pad1)
- U341 pad 7: Net-(C345-Pad1) -> /DAC2752-2A/Force
- U342 pad 2: Net-(U341-S1) -> /DAC2752-2A/Sense
- U35 pad 28: Net-(U35B-IOUT2BF) -> /DAC2752-2B/IOUT2
- U35 pad 29: Net-(U35B-IOUT2BF) -> Net-(U35B-IOUT2BS)
- U35 pad 31: Net-(C372-Pad1) -> /DAC2752-2B/RSense
- U35 pad 32: Net-(U36B--) -> /DAC2752-2B/RIN
- U35 pad 34: Net-(U35B-RCOMB) -> /DAC2752-2B/RCOM
- U35 pad 35: Net-(C362-Pad1) -> /DAC2752-2B/FREF
- U35 pad 36: Net-(C362-Pad1) -> /DAC2752-2B/FREF
- U35 pad 39: Net-(U361-S1) -> /DAC2752-2B/RFB
- U35 pad 40: Net-(C363-Pad1) -> /DAC2752-2B/Sense
- U35 pad 41: Net-(U35B-IOUT1B) -> /DAC2752-2B/IOUT1
- U35 pad 44: Net-(U35A-IOUT1A) -> /DAC2752-2A/IOUT1
- U35 pad 45: Net-(C343-Pad1) -> /DAC2752-2A/Sense
- U35 pad 46: Net-(U341-S1) -> /DAC2752-2A/RFB
- U35 pad 8: Net-(U35A-IOUT2AF) -> Net-(U35A-IOUT2AS)
- U35 pad 9: Net-(U35A-IOUT2AF) -> /DAC2752-2A/IOUT2
- U36 pad 6: Net-(U36B--) -> /DAC2752-2B/RSense
- U36 pad 7: Net-(C372-Pad1) -> /DAC2752-2B/RIN
- U361 pad 1: Net-(C362-Pad1) -> /DAC2752-2B/Force
- U361 pad 2: Net-(U304A--) -> Net-(U361A--)
- U361 pad 6: Net-(U304B--) -> Net-(U361B--)
- U361 pad 7: Net-(C366-Pad1) -> /DAC2752-2B/FREF
- U362 pad 2: Net-(U361-S1) -> /DAC2752-2B/Sense
- U37 pad 5: Net-(U35A-IOUT1A) -> /DAC2752-2A/IOUT1
- U38 pad 1: Net-(C361-Pad1) -> Net-(C364-Pad1)
- U38 pad 3: Net-(U35B-RCOMB) -> /DAC2752-2B/IOUT1
- U38 pad 5: Net-(U35B-IOUT1B) -> /DAC2752-2B/RCOM
- U38 pad 7: Net-(C364-Pad1) -> Net-(C361-Pad1)
- U43 pad 4: Net-(U43-ILIM) -> /Low Voltage Power/I6V
- U43 pad 6: Net-(U43-EN) -> /Low Voltage Power/I6V
- U43 pad 8: Net-(U43-EN) -> /Low Voltage Power/I6V
- U706 pad 3: /FDA/Out- -> /FDA/IN+
- U706 pad 5: /FDA/IN+ -> /FDA/Out-
- U707 pad 1: Net-(R744-Pad1) -> Net-(C743-Pad2)
- U707 pad 3: /FDA/Out+ -> GND
- U707 pad 5: GND -> /FDA/Out+
- U707 pad 7: Net-(R749-Pad1) -> Net-(C745-Pad2)
Routing:
- net +18V: track 0.00 -> 185.8 mm, vias 0 -> 12
- net -18V: track 0.00 -> 105.6 mm, vias 0 -> 8
- net GNDPWR: track 57.2 -> 154.9 mm, vias 20 -> 96
- net +2V5: track 0.00 -> 70.3 mm, vias 0 -> 4
- net GND: track 0.00 -> 65.8 mm, vias 0 -> 24
- net /~{LDAC}: track 0.00 -> 63.3 mm, vias 0 -> 4
- net -2V5: track 0.00 -> 55.3 mm, vias 0 -> 6
- net Net-(U27-S1): track 0.00 -> 55.3 mm, vias 0 -> 8
- net /MISO: track 0.00 -> 40.1 mm, vias 0 -> 4
- net /SCK: track 0.00 -> 38.0 mm, vias 0 -> 4
- net /MOSI: track 0.00 -> 34.6 mm, vias 0 -> 2
- net /Sample Hold 2/Drive: track 0.00 -> 33.9 mm
- net /Comp1B: track 0.00 -> 31.7 mm, vias 0 -> 2
- net /DAC2752-2A/FREF: track 0.00 -> 26.9 mm, vias 0 -> 2
- net /DAC2752-1B/FREF: track 0.00 -> 26.7 mm, vias 0 -> 2
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- added copper zone on In2.Cu, net GND

Commit message: Tweaks following spice simulation.
Parts:
- removed C67, C741: 10u, Capacitor_SMD:C_0603_1608Metric
- removed C68: 1u, Capacitor_SMD:C_0402_1005Metric
- removed C737: 0u1, Capacitor_SMD:C_0402_1005Metric
- removed C738, C739, C740: 10n, Capacitor_SMD:C_0603_1608Metric
- removed C742, C743, C744, C745: 0n1, Capacitor_SMD:C_0402_1005Metric
- removed C761, C762, C763, C765, C766: 1n, Capacitor_SMD:C_0603_1608Metric
- removed J61, J62: Conn_01x01_Socket, TestPoint:TestPoint_Plated_Hole_D5.0mm
- removed JP703: SolderJumper_2_Open, Parts:ThermJump_1
- removed JP704: SolderJumper_2_Bridged, Parts:ThermJumpBridge
- removed L63, L75, L76: 100, Inductor_SMD:L_0603_1608Metric
- removed R120, R121: 0R33, Resistor_SMD:R_0805_2012Metric
- removed R461: 1, Resistor_SMD:R_0603_1608Metric
- removed R739, R740, R747, R748: 100k, Resistor_SMD:R_0402_1005Metric
- removed R741, R746, R749, R753, R754: 10k, Resistor_SMD:R_0402_1005Metric
- removed R742, R744, R750: 1k2, Resistor_SMD:R_0402_1005Metric
- removed R743, R745, R751: 62k, Resistor_SMD:R_0603_1608Metric
- removed R752: 100, Resistor_SMD:R_0603_1608Metric
- removed R761, R763, R764: 470, Resistor_SMD:R_0402_1005Metric
- removed R762, R765: 330, Resistor_SMD:R_0402_1005Metric
- removed U707: OPA2197D, Parts:OPA2197
- added C316: 10u, Capacitor_SMD:C_0603_1608Metric, F.Cu at (286.4, 181.8)
- added C334: 10u, Capacitor_SMD:C_0603_1608Metric, F.Cu at (303.5, 180.2)
- added C355: 10u, Capacitor_SMD:C_0603_1608Metric, F.Cu at (286.5, 144.8)
- added C375: 10u, Capacitor_SMD:C_0603_1608Metric, F.Cu at (303.5, 143.2)
- added C401: 10u, Capacitor_SMD:C_0603_1608Metric, F.Cu at (147.8, 119.4)
- added C411: 10u, Capacitor_SMD:C_0603_1608Metric, F.Cu at (152.9, 140.0)
- added C421: 10u, Capacitor_SMD:C_0603_1608Metric, F.Cu at (150.9, 150.3)
- added C468: 10u, Capacitor_SMD:C_0603_1608Metric, F.Cu at (145.7, 162.3)
- added C551: 10u, Capacitor_SMD:C_0805_2012Metric, F.Cu at (166.6, 203.2)
- added C724: 0n1, Capacitor_SMD:C_0603_1608Metric, F.Cu at (226.2, 92.5)
- added C779: 10u, Capacitor_SMD:C_0603_1608Metric, F.Cu at (245.3, 116.7)
- added C854: 10u, Capacitor_SMD:C_0603_1608Metric, F.Cu at (81.2, 186.4)
- added D42: 1N5819WS, Diode_SMD:D_SOD-323, F.Cu at (148.6, 142.6)
- added D55: 1N5819WS, Diode_SMD:D_SOD-323, F.Cu at (148.6, 181.5)
- added D56: 1N5819WS, Diode_SMD:D_SOD-323, F.Cu at (151.3, 194.7)
- added JP71: SolderJumper_2_Bridged, Parts:JumperClosed, F.Cu at (199.8, 93.5)
- added L401: 600, Inductor_SMD:L_0603_1608Metric, F.Cu at (147.3, 116.7)
- added L411: 600, Inductor_SMD:L_0603_1608Metric, F.Cu at (150.3, 136.8)
- added L421: 600, Inductor_SMD:L_0603_1608Metric, F.Cu at (150.1, 146.5)
- added L461: 600, Inductor_SMD:L_0603_1608Metric, F.Cu at (142.5, 159.0)
- added L56: 600, Inductor_SMD:L_0603_1608Metric, F.Cu at (162.8, 201.4)
- added L83: 600, Inductor_SMD:L_0603_1608Metric, F.Cu at (85.5, 185.2)
- added R316: 100, Resistor_SMD:R_0603_1608Metric, F.Cu at (290.5, 198.1)
- added R336: 100, Resistor_SMD:R_0603_1608Metric, F.Cu at (299.5, 198.1)
- added R356: 100, Resistor_SMD:R_0603_1608Metric, F.Cu at (290.5, 161.1)
- added R376: 100, Resistor_SMD:R_0603_1608Metric, F.Cu at (299.5, 161.1)
- added R63: 1, Resistor_SMD:R_0603_1608Metric, F.Cu at (140.0, 87.2)
- added R714: 10, Resistor_SMD:R_0402_1005Metric, F.Cu at (284.2, 73.6)
- added TP62: TestPoint, Parts:TestPoint, F.Cu at (130.7, 72.0)
- added TP63: TestPoint, Parts:TestPoint, F.Cu at (130.7, 74.3)
- C101, C102: value 1u -> 10n; footprint Capacitor_SMD:C_0402_1005Metric -> Capacitor_SMD:C_0603_1608Metric
- C104, C116, C305, C307, C308, C321, C322, C327, C346, C347, C348, C365, C367, C368, C381, C383, C465, C718, C719, C732, C83, C851, C852: value 0u1 -> 1u
- C404: renamed from C403; value 0u1 -> 1u
- C414: renamed from C413; value 0u1 -> 1u
- C424: renamed from C425; value 0u1 -> 1u
- C433: renamed from C435; value 0u1 -> 1u
- C720, C721: value 0n1 -> 3n3
- C722: value 330p -> 0n1
- C723: value 1n -> 0n1
- C725: value 1n -> 10u
- C726: value 1n -> 470n; footprint Capacitor_SMD:C_0603_1608Metric -> Capacitor_SMD:C_0402_1005Metric
- C727, C760, C764: value 1n -> 10n
- C729, C730: value 10n -> 10p; footprint Capacitor_SMD:C_0603_1608Metric -> Capacitor_SMD:C_0402_1005Metric
- C731: value 10n -> 1u; footprint Capacitor_SMD:C_0603_1608Metric -> Capacitor_SMD:C_0402_1005Metric
- C733, C735: value 0u1 -> 10u; footprint Capacitor_SMD:C_0402_1005Metric -> Capacitor_SMD:C_0603_1608Metric
- C911: renamed from C724; value 330p -> 22p
- J1: renamed from J71; footprint TestPoint:TestPoint_Plated_Hole_D5.0mm -> Parts:Plated_Hole_D4.0mm_10mm
- J2: renamed from J72; footprint TestPoint:TestPoint_Plated_Hole_D5.0mm -> Parts:Plated_Hole_D4.0mm_10mm
- J3: renamed from J73; footprint TestPoint:TestPoint_Plated_Hole_D5.0mm -> Parts:Plated_Hole_D4.0mm_10mm
- J4: renamed from J74; footprint TestPoint:TestPoint_Plated_Hole_D5.0mm -> Parts:Plated_Hole_D4.0mm_10mm
- J5: renamed from J75; footprint TestPoint:TestPoint_Plated_Hole_D5.0mm -> Parts:Plated_Hole_D4.0mm_10mm
- J6: renamed from J76; footprint TestPoint:TestPoint_Plated_Hole_D5.0mm -> Parts:Plated_Hole_D4.0mm_10mm
- JP21, JP22: footprint Parts:ThermJump_1 -> Parts:JumperOpen
- L54, L55: value 100 -> 600
- NT61: footprint NetTie:NetTie-2_SMD_Pad0.5mm -> Parts:NetTie-2_SMD_Pad0.5mm
- R315, R335, R355, R375: footprint Resistor_SMD:R_0402_1005Metric -> Resistor_SMD:R_0603_1608Metric
- R462: value 11k -> 20k; footprint Resistor_SMD:R_0603_1608Metric -> Resistor_SMD:R_0402_1005Metric
- R463: value 10k -> 24k; footprint Resistor_SMD:R_0402_1005Metric -> Resistor_SMD:R_0603_1608Metric
- R464: value 390k -> 68k
- R61: renamed from R65; footprint Resistor_SMD:R_0402_1005Metric_Pad0.72x0.64mm_HandSolder -> Resistor_SMD:R_0603_1608Metric
- R62: renamed from R66; footprint Resistor_SMD:R_0402_1005Metric_Pad0.72x0.64mm_HandSolder -> Resistor_SMD:R_0603_1608Metric
- R67: footprint Resistor_SMD:R_0603_1608Metric -> Resistor_SMD:R_0402_1005Metric
- R713: value 10M -> 100; footprint Resistor_SMD:R_0603_1608Metric -> Resistor_SMD:R_0402_1005Metric
- R720: value 0 -> 1k; footprint Resistor_SMD:R_0603_1608Metric -> Capacitor_SMD:C_0402_1005Metric
- R721: value 240 -> 1k; footprint Resistor_SMD:R_0603_1608Metric -> Capacitor_SMD:C_0402_1005Metric
- R722: value 240 -> 1k2; footprint Resistor_SMD:R_0603_1608Metric -> Capacitor_SMD:C_0603_1608Metric
- R723: value 24k -> 1k2; footprint Resistor_SMD:R_0603_1608Metric -> Capacitor_SMD:C_0603_1608Metric
- R724: value 24k -> 10; footprint Resistor_SMD:R_0603_1608Metric -> Resistor_SMD:R_0402_1005Metric
- R725: value 240 -> 10; footprint Resistor_SMD:R_0603_1608Metric -> Resistor_SMD:R_0402_1005Metric
- R726: value 240 -> 10k
- R727: value 750 -> 10k
- R728, R729: value 100 -> 10k; footprint Resistor_SMD:R_0603_1608Metric -> Resistor_SMD:R_0402_1005Metric
- R731: value 100 -> 10k
- R732: value 1 -> 100k; footprint Resistor_SMD:R_0603_1608Metric -> Resistor_SMD:R_0402_1005Metric
- R733: value 1 -> 1k5; footprint Resistor_SMD:R_0603_1608Metric -> Resistor_SMD:R_0402_1005Metric
- R734: value 10k -> 12k; footprint Resistor_SMD:R_0402_1005Metric_Pad0.72x0.64mm_HandSolder -> Resistor_SMD:R_0603_1608Metric
- R735: value 10k -> 100k; footprint Resistor_SMD:R_0402_1005Metric_Pad0.72x0.64mm_HandSolder -> Resistor_SMD:R_0402_1005Metric
- R736: value 62k -> 10k; footprint Resistor_SMD:R_0603_1608Metric -> Resistor_SMD:R_0402_1005Metric
- R737: value 1k2 -> 1k5
- R738: value 10k -> 12k; footprint Resistor_SMD:R_0402_1005Metric -> Resistor_SMD:R_0603_1608Metric
- R760: value 470 -> 100
- RN61, RN71, RN72, RN73, RN81: footprint Package_SO:MSOP-8-1EP_3x3mm_P0.65mm_EP1.68x1.88mm -> Parts:MSOP-8-1EP_3x3mm_P0.65mm_EP1.68x1.88mm
- U74: value THS4521IDGK -> THS4541IDGK; footprint Parts:MSOP-8_3x3mm_P0.65mm -> Parts:OPA4521
- moved C778 104.7 mm to (258.1, 100.6), turned to 90 degrees
- moved C760 103.6 mm to (249.6, 115.8)
- moved C768 102.9 mm to (253.2, 117.5)
- moved C770 100.9 mm to (253.4, 115.4)
- moved L79 100.5 mm to (253.2, 119.5)
- moved L80 100.5 mm to (253.2, 122.0)
- moved C771 100.3 mm to (250.2, 102.1)
- moved C772 100.1 mm to (247.3, 111.0), turned to 180 degrees
- moved C777 99.9 mm to (258.4, 105.2)
- moved C769 99.8 mm to (248.8, 102.5), turned to -90 degrees
- moved L77 99.6 mm to (258.4, 106.7), turned to 180 degrees
- moved C773 99.3 mm to (245.3, 115.5), turned to 180 degrees
- moved C767 98.9 mm to (247.3, 102.1), turned to 180 degrees
- moved C774 97.3 mm to (251.2, 93.4)
- moved R703 95.5 mm to (191.1, 105.5)
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- renumbered C401 to C402, C402 to C403, C404 to C405, C405 to C406, C406 to C407, C411 to C412, C412 to C413, C414 to C415, C415 to C416, C416 to C417, C421 to C422, C422 to C423, C423 to C425, C424 to C426, C426 to C427, C433 to C434, C434 to C435, C542 to C541, C543 to C542, C544 to C543, C545 to C544, C546 to C545, C547 to C546, C548 to C547, C549 to C548, C550 to C549, C551 to C550, D42 to D43, J85 to J7, L41 to L40, L42 to L41, L43 to L42, L44 to L43, L47 to L44, L48 to L47, R61 to R64, R62 to R65, R64 to R66
Connections:
- net Net-(C716-Pad2) renamed /Monitor/BufA
- net Net-(C717-Pad2) renamed /Monitor/BufB
- net Net-(U76A--) renamed /Monitor/FbA
- net Net-(U76B--) renamed /Monitor/FbB
- net Net-(U77A-+) renamed /Monitor/Vg
- C464 pad 1: Net-(U45-FB) -> Net-(C464-Pad1)
- C464 pad 2: -2V5 -> Net-(U45-FB)
- C465 pad 2: -2V5 -> Net-(C464-Pad1)
- C466 pad 1: -2V5 -> Net-(C464-Pad1)
- C467 pad 1: -2V5 -> Net-(C464-Pad1)
- C544 pad 2: -18V -> Net-(C544-Pad2)
- C545 pad 2: -18V -> Net-(C544-Pad2)
- C546 pad 2: -18V -> Net-(C544-Pad2)
- C547 pad 2: -18V -> Net-(C544-Pad2)
- C548 pad 2: -18V -> Net-(C544-Pad2)
- C549 pad 2: -18V -> Net-(C544-Pad2)
- C703 pad 1: Net-(JP704-A) -> /Monitor/Isum
- C705 pad 2: Net-(JP704-A) -> /Monitor/Isum
- C720 pad 1: Net-(U74-+) -> /ADC-
- C720 pad 2: Net-(C720-Pad2) -> GNDPWR
- C721 pad 1: Net-(C721-Pad1) -> GNDPWR
- C721 pad 2: Net-(U74--) -> /ADC+
- C722 pad 1: Net-(C722-Pad1) -> Net-(U74-+)
- C722 pad 2: GNDPWR -> Net-(C722-Pad2)
- C723 pad 1: Net-(C722-Pad1) -> Net-(C723-Pad1)
- C723 pad 2: GNDPWR -> Net-(U74--)
- C725 pad 1: Net-(C724-Pad1) -> Net-(C725-Pad1)
- C725 pad 2: Net-(U73A--) -> GNDPWR
- C726 pad 1: Net-(C726-Pad1) -> /FDA/ForceCM
- C726 pad 2: Net-(U73A-+) -> GNDPWR
- C727 pad 2: Net-(U73A--) -> /FDA/SenseCM
- C728 pad 1: Net-(C728-Pad1) -> Ref2V5
- C729 pad 2: GNDPWR -> Net-(U706A--)
- C730 pad 1: /FDA/Out- -> Net-(U706B--)
- C730 pad 2: /FDA/Out+ -> Net-(C730-Pad2)
- C731 pad 1: Net-(U74-V_{OCM}) -> +5VA
- C732 pad 1: +18V -> +5VA
- C733 pad 1: GNDPWR -> +5VA
- C733 pad 2: -18V -> GNDPWR
- C734 pad 1: +5VA -> +18V
- C735 pad 1: +5VA -> GNDPWR
- C735 pad 2: GNDPWR -> -2V5
- C736 pad 1: +18V -> GNDPWR
- C736 pad 2: GNDPWR -> -18V
- C760 pad 1: Net-(U75A-+) -> Net-(U75B-+)
- C764 pad 1: Net-(U75B-+) -> Ref0V
- C772 pad 1: GNDPWR -> +18V
- C772 pad 2: +18V -> GNDPWR
- C773 pad 1: -2V5 -> GNDPWR
- C773 pad 2: GNDPWR -> -2V5
- C851 pad 1: +5VA -> Net-(U85-VDD)
- C911 pad 1: Net-(C724-Pad1) -> /FDA/Stage1
- C911 pad 2: Net-(U73A--) -> /FDA/In-Fb+
- D71 pad 1: GNDPWR -> +5VA
- D71 pad 2: Net-(D71-A) -> /Monitor ADC/BufR+
- D72 pad 1: Net-(D71-A) -> /Monitor ADC/BufR+
- D73 pad 1: +5VA -> GNDPWR
- D73 pad 2: Net-(D73-A) -> /Monitor ADC/BufR-
- D74 pad 1: Net-(D73-A) -> /Monitor ADC/BufR-
- J5 pad 1: Net-(J75-Pin_1) -> Net-(J5-Pin_1)
- L11 pad 2: Net-(L11-Pad2) -> Net-(U19C-VCC)
- L12 pad 2: Net-(L12-Pad2) -> Net-(C111-Pad2)
- L40 pad 2: /Low Voltage Power/I5VA -> Net-(C401-Pad1)
- L41 pad 2: /Low Voltage Power/I3V3A -> Net-(C411-Pad1)
- L42 pad 2: /Low Voltage Power/I2V5 -> Net-(C421-Pad1)
- L44 pad 2: Net-(L47-Pad2) -> Net-(U45-EN)
- R462 pad 1: -2V5 -> Net-(C464-Pad1)
- R541 pad 1: -18V -> Net-(C544-Pad2)
- R62 pad 2: GND -> Ref0V
- R707 pad 1: Net-(U78B--) -> Net-(U78A--)
- R708 pad 2: Net-(U78B--) -> Net-(U78A--)
- R713 pad 1: Net-(U78A-+) -> Net-(JP71-B)
- R713 pad 2: GNDPWR -> Net-(J5-Pin_1)
- R720 pad 1: Net-(R720-Pad1) -> Net-(U74-+)
- R720 pad 2: Net-(C724-Pad1) -> /FDA/Stage1
- R721 pad 1: Net-(U74-+) -> Net-(U74--)
- R721 pad 2: Net-(R720-Pad1) -> Net-(C725-Pad1)
- R722 pad 1: Net-(U74--) -> /FDA/Force-
- R722 pad 2: Net-(C741-Pad1) -> Net-(C722-Pad2)
- R723 pad 1: /FDA/Out- -> /FDA/Force+
- R723 pad 2: Net-(U74-+) -> Net-(C723-Pad1)
- R724 pad 1: /FDA/Out+ -> /ADC-
- R724 pad 2: Net-(U74--) -> /FDA/Force-
- R725 pad 1: Net-(R725-Pad1) -> /ADC+
- R725 pad 2: Net-(C720-Pad2) -> /FDA/Force+
- R726 pad 1: Net-(R726-Pad1) -> /ADC-
- R726 pad 2: Net-(C721-Pad1) -> /FDA/SenseCM
- R727 pad 1: Net-(C722-Pad1) -> /FDA/SenseCM
- R727 pad 2: Net-(U73A-+) -> /ADC+
- R728 pad 1: Net-(R725-Pad1) -> Net-(C725-Pad1)
- R728 pad 2: Net-(C726-Pad1) -> +5VA
- R729 pad 1: Net-(R726-Pad1) -> Net-(C725-Pad1)
- R729 pad 2: Net-(C727-Pad1) -> GNDPWR
- R730 pad 1: /FDA/Out- -> /FDA/ForceCM
- R730 pad 2: Net-(R725-Pad1) -> Net-(C727-Pad1)
- R731 pad 1: /FDA/Out+ -> Net-(C729-Pad1)
- R731 pad 2: Net-(R726-Pad1) -> Net-(U706A--)
- R732 pad 1: /FDA/Out- -> Net-(U706A--)
- R732 pad 2: Net-(C728-Pad1) -> /Sum+
- R733 pad 2: /FDA/Out+ -> /ADC-
- R734 pad 1: /FDA/Out- -> Net-(C729-Pad1)
- R734 pad 2: Net-(U73B--) -> /ADC-
- R735 pad 1: Net-(U73B--) -> Net-(U706B--)
- R735 pad 2: /FDA/Out+ -> /Sum-
- R736 pad 1: Net-(C742-Pad1) -> Net-(U706B--)
- R736 pad 2: /FDA/IN+ -> Net-(C730-Pad2)
- R737 pad 1: Net-(C742-Pad1) -> Net-(C730-Pad2)
- R737 pad 2: /FDA/IN+ -> /ADC+
- R738 pad 1: Net-(C742-Pad1) -> Net-(C730-Pad2)
- R738 pad 2: Net-(U706A--) -> /ADC+
- R760 pad 1: GND -> Ref5V
- R760 pad 2: Net-(U75A-+) -> Net-(U75B-+)
- RN71 pad 2: Net-(JP704-A) -> /Monitor/Isum
- RN72 pad 1: Net-(U73A-+) -> /ADC-
- RN72 pad 2: /FDA/IN+ -> /FDA/In+Fb-
- RN72 pad 3: /FDA/Out- -> /FDA/In+Fb-
- RN72 pad 4: Net-(U73A-+) -> /ADC-
- RN72 pad 5: /FDA/Out- -> /FDA/In+Fb-
- RN72 pad 6: Net-(U73A-+) -> /ADC-
- RN72 pad 7: Net-(U73A-+) -> /Sum+
- RN72 pad 8: /FDA/Out- -> /FDA/In+Fb-
- RN73 pad 1: Net-(U73A--) -> /ADC+
- RN73 pad 2: /FDA/Out+ -> /FDA/In-Fb+
- RN73 pad 3: GND -> /FDA/In-Fb+
- RN73 pad 4: Net-(U73A--) -> /ADC+
- RN73 pad 5: /FDA/Out+ -> /FDA/In-Fb+
- RN73 pad 6: Net-(U73A--) -> /Sum-
- RN73 pad 7: Net-(U73A--) -> /ADC+
- RN73 pad 8: /FDA/Out+ -> /FDA/In-Fb+
- TP54 pad 1: -18V -> Net-(C544-Pad2)
- U45 pad 1: -2V5 -> Net-(C464-Pad1)
- U45 pad 20: -2V5 -> Net-(C464-Pad1)
- U53 pad 1: -18V -> Net-(C544-Pad2)
- U53 pad 20: -18V -> Net-(C544-Pad2)
- U7 pad 1: Net-(D71-A) -> /ADC+
- U7 pad 2: Net-(D71-A) -> /Monitor ADC/BufR-
- U7 pad 21: /FDA/Out- -> unconnected-(U7-AIN0-Pad21)
- U7 pad 22: /FDA/Out+ -> /Monitor ADC/BufR+
- U7 pad 23: GNDPWR -> /Monitor ADC/BufR-
- U7 pad 24: Net-(D73-A) -> /ADC-
- U7 pad 3: Net-(D73-A) -> /Monitor ADC/BufR+
- U706 pad 1: Net-(C742-Pad1) -> Net-(C729-Pad1)
- U706 pad 3: /FDA/IN+ -> /ADC-
- U706 pad 5: /FDA/Out- -> /ADC+
- U706 pad 7: Net-(C744-Pad1) -> Net-(C730-Pad2)
- U73 pad 1: Net-(R720-Pad1) -> /FDA/Stage1
- U73 pad 2: Net-(U73A--) -> /FDA/In-Fb+
- U73 pad 3: Net-(U73A-+) -> /FDA/In+Fb-
- U73 pad 6: Net-(U73B--) -> /FDA/SenseCM
- U73 pad 7: Net-(C738-Pad1) -> Net-(C727-Pad1)
- U74 pad 2: Net-(U74-V_{OCM}) -> /FDA/ForceCM
- U74 pad 4: Net-(R726-Pad1) -> /FDA/Force+
- U74 pad 5: Net-(R725-Pad1) -> /FDA/Force-
- U75 pad 1: Net-(C761-Pad2) -> /Monitor ADC/BufR-
- U75 pad 2: Net-(U75A--) -> /Monitor ADC/BufR-
- U75 pad 3: Net-(U75A-+) -> Ref0V
- U75 pad 6: Net-(U75B--) -> /Monitor ADC/BufR+
- U75 pad 7: Net-(C765-Pad2) -> /Monitor ADC/BufR+
- U77 pad 5: GNDPWR -> GND
- U77 pad 6: Net-(U77B--) -> /Sum-
- U77 pad 7: Net-(U77B--) -> /Sum-
- U78 pad 1: Net-(JP703-A) -> /Monitor/Isum
- U78 pad 2: Net-(JP703-A) -> Net-(U78A--)
- U78 pad 3: Net-(U78A-+) -> GND
- U78 pad 5: GND -> Net-(JP71-B)
- U78 pad 6: Net-(U78B--) -> /Sum+
- U78 pad 7: Net-(JP704-A) -> /Sum+
- U81 pad 1: /SHSample1 -> /SHSampleG2
- U81 pad 15: /SHOutEn1 -> /SHHoldG2
- U81 pad 2: /SHSampleG1 -> /SHSample2
- U81 pad 3: /SHHoldG1 -> /SHOutEn2
- U81 pad 4: /SHOutEn2 -> /SHHoldG1
- U81 pad 5: /SHSample2 -> /SHSampleG1
- U81 pad 6: /SHSampleG2 -> /SHSample1
- U81 pad 7: /SHHoldG2 -> /SHOutEn1
- U82 pad 1: /OffsetA1 -> /MonB0
- U82 pad 15: /OffsetA0 -> /MonB1
- U82 pad 2: /OffsetA2 -> /MonA1
- U82 pad 3: /SHSel -> /MonA0
- U82 pad 4: /MonA0 -> /SHSel
- U82 pad 5: /MonA1 -> /OffsetA2
- U82 pad 6: /MonB0 -> /OffsetA1
- U82 pad 7: /MonB1 -> /OffsetA0
- U83 pad 1: /Sel1B -> unconnected-(U83-QB-Pad1)
- U83 pad 15: /Sel1A -> unconnected-(U83-QA-Pad15)
- U83 pad 2: /Sel2A -> unconnected-(U83-QC-Pad2)
- U83 pad 3: /Sel2B -> unconnected-(U83-QD-Pad3)
- U83 pad 4: unconnected-(U83-QE-Pad4) -> /Sel2B
- U83 pad 5: unconnected-(U83-QF-Pad5) -> /Sel2A
- U83 pad 6: unconnected-(U83-QG-Pad6) -> /Sel1B
- U83 pad 7: unconnected-(U83-QH-Pad7) -> /Sel1A
- U85 pad 7: +5VA -> Net-(U85-VDD)
Routing:
- net /ADC+: track 0.00 -> 100.1 mm, vias 0 -> 4
- net /ADC-: track 0.00 -> 91.7 mm, vias 0 -> 5
- net /Sum-: track 0.00 -> 80.2 mm, vias 0 -> 5
- net /Sum+: track 0.00 -> 78.6 mm, vias 0 -> 5
- net +18V: track 185.8 -> 248.9 mm, vias 12 -> 17
- net -18V: track 105.6 -> 158.1 mm, vias 8 -> 13
- net /Monitor ADC/BufR+: track 0.00 -> 50.6 mm, vias 0 -> 1
- net /Monitor ADC/BufR-: track 0.00 -> 49.6 mm, vias 0 -> 1
- net /FDA/In-Fb+: track 0.00 -> 40.5 mm, vias 0 -> 4
- net /FDA/In+Fb-: track 0.00 -> 40.5 mm, vias 0 -> 4
- net /FDA/SenseCM: track 0.00 -> 30.3 mm, vias 0 -> 2
- net GNDPWR: track 154.9 -> 183.3 mm, vias 96 -> 122
- net /Monitor/BufA: track 0.00 -> 27.9 mm, vias 0 -> 1
- net /Monitor/BufB: track 0.00 -> 27.8 mm, vias 0 -> 2
- net /Monitor/Isum: track 0.00 -> 26.1 mm, vias 0 -> 4
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