File: lincal.kicad_pcb (KiCad board)
At the start: 4 copper layers, 250 x 150 mm, 554 parts, among them J1 Conn_01x01_Socket, J2 Conn_01x01_Socket, J3 Conn_01x01_Socket, J4 Conn_01x01_Socket, J5 Conn_01x01_Socket, J6 Conn_01x01_Socket, J7 USB_C_Receptacle_USB2.0_16P, J81 Conn_01x03_Pin, J82 Conn_Coaxial, J83 Conn_Coaxial, J84 Conn_01x02_Pin, J86 Conn_01x02_Pin, Q81 Si2301CDS, Q82 AO3400A, SW81 SW_Push, SW82 SW_Push, U11 OPA2189DGK, U12 TMUX1108PW, U30 LTC2752B, U301 OPA2197D, U302 DG419D, U31 OPA2189DGK, U32 OPA2388DGK, U321 OPA2197D, U322 DG419D, U33 OPA2388DGK, U341 OPA2197D, U342 DG419D, U35 LTC2752B, U36 OPA2189DGK, U361 OPA2197D, U362 DG419D, U37 OPA2388DGK, U38 OPA2388DGK, U41 TPS7A8801RTJR, U42 TPS7A8801RTJR, U43 TPS61252DSG, U44 TPSM863252RDXR, U45 TPS7A3301RGW, U46 TPSM863252RDXR, U51 ADP5071ACPZ, U52 TPS7A4700xRGW, U53 TPS7A3301RGW, U6 REF7050, U61 OPA2189DGK, U7 AD7177-2BRUZ, U70 TG2520SMN-16M-MCG, U704 OPA2197D, U706 OPA2197D, U71 TMUX6104, U72 TMUX6104, U73 OPA2388DGK, U74 THS4521IDGK, U75 OPA2189DGK, U76 OPA2189DGK, U77 OPA2388DGK, U78 OPA2189DGK, U8 ESP32-C6-MINI-1U, U81 74HC595, U82 74HC595, U84 ISOW7842, U85 DAC80508xRTE

Commit message: Most blocks there....
About to restore scan.
Parts:
- removed C313, C326, C352, C372: 0n1, Capacitor_SMD:C_0402_1005Metric
- removed C316, C334, C355, C375: 10u, Capacitor_SMD:C_0603_1608Metric
- removed C550: 10u, Capacitor_SMD:C_0805_2012Metric
- removed NT31, NT32, NT33, NT34: NetTie_2, Parts:NetTie-2_SMD_Pad0.5mm
- removed R305, R325, R345, R365: 2k4, Resistor_SMD:R_0402_1005Metric
- removed R306, R326, R346, R366: 1k2, Resistor_SMD:R_0402_1005Metric
- removed R307, R314, R327, R334, R347, R354, R367, R374: 1k, Resistor_SMD:R_0402_1005Metric
- removed R308, R313, R328, R333, R348, R353, R368, R373: 0, Resistor_SMD:R_0603_1608Metric
- removed R544: 1, Resistor_SMD:R_0603_1608Metric
- removed TP301, TP302, TP303, TP304, TP321, TP322, TP323, TP324, TP341, TP342, TP343, TP344, TP361, TP362, TP363, TP364: TestPoint, Parts:TestPoint
- added C387: 1u, Capacitor_SMD:C_0402_1005Metric, F.Cu at (303.4, 191.4)
- added C388: 1u, Capacitor_SMD:C_0402_1005Metric, F.Cu at (305.1, 186.9)
- added C389: 1u, Capacitor_SMD:C_0402_1005Metric, F.Cu at (303.4, 154.4)
- added C390: 1u, Capacitor_SMD:C_0402_1005Metric, F.Cu at (305.1, 149.9)
- added R119: 100, Resistor_SMD:R_0402_1005Metric, F.Cu at (0.95, 0.49)
- added U34: OPA2388DGK, Parts:OPA2388, F.Cu at (304.3, 189.2)
- added U39: OPA2388DGK, Parts:OPA2388, F.Cu at (304.3, 152.2)
- R83: footprint Resistor_SMD:R_0603_1608Metric -> Resistor_SMD:R_0402_1005Metric
- moved C551 38.0 mm to (130.5, 191.4)
- moved L56 32.6 mm to (131.0, 193.9), turned to -90 degrees
- moved C468 17.5 mm to (130.2, 170.6)
- moved L461 16.0 mm to (129.5, 168.3), turned to 90 degrees
- moved TP51 7.55 mm to (121.2, 182.6)
- moved C527 5.35 mm to (147.2, 186.2)
- moved C528 5.35 mm to (150.7, 186.2)
- moved C529 5.35 mm to (141.8, 186.1)
- moved C530 5.35 mm to (144.8, 186.1)
- moved C526 4.25 mm to (135.1, 187.7)
- moved C525 4.15 mm to (137.3, 186.2)
- moved C523 4.10 mm to (131.9, 187.2), turned to -90 degrees
- moved U52 4.10 mm to (134.1, 183.6)
- moved C524 4.05 mm to (130.1, 184.2)
- moved C522 4.05 mm to (130.3, 187.0), turned to -90 degrees
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- renumbered C507 to C50, C501 to C51, C504 to C52, C506 to C53
Connections:
- net Net-(U6-EN) renamed /Reference/rin
- C461 pad 1: Net-(U45-EN) -> /Low Voltage Power/Im2V5
- C462 pad 1: Net-(U45-EN) -> /Low Voltage Power/Im2V5
- C464 pad 1: Net-(C464-Pad1) -> -2V5
- C465 pad 2: Net-(C464-Pad1) -> -2V5
- C466 pad 1: Net-(C464-Pad1) -> -2V5
- C467 pad 1: Net-(C464-Pad1) -> -2V5
- C468 pad 1: -2V5 -> Net-(C468-Pad1)
- C52 pad 1: GNDPWR -> Net-(D51-K)
- C52 pad 2: Net-(D51-K) -> GNDPWR
- C522 pad 1: GNDPWR -> /18V/i18
- C522 pad 2: Net-(U52-EN) -> GNDPWR
- C523 pad 1: GNDPWR -> /18V/i18
- C523 pad 2: Net-(U52-EN) -> GNDPWR
- C53 pad 1: Net-(D52-A) -> GNDPWR
- C53 pad 2: GNDPWR -> Net-(D52-A)
- C541 pad 1: Net-(U53-EN) -> /18V/im18
- C542 pad 1: Net-(U53-EN) -> /18V/im18
- C543 pad 1: GNDPWR -> Net-(U53-NR/SS)
- C543 pad 2: Net-(U53-NR/SS) -> GNDPWR
- C544 pad 1: GNDPWR -> -18V
- C544 pad 2: Net-(C544-Pad2) -> GNDPWR
- C545 pad 1: Net-(U53-FB) -> -18V
- C545 pad 2: Net-(C544-Pad2) -> Net-(U53-FB)
- C546 pad 1: GNDPWR -> -18V
- C546 pad 2: Net-(C544-Pad2) -> GNDPWR
- C547 pad 1: GNDPWR -> -18V
- C547 pad 2: Net-(C544-Pad2) -> GNDPWR
- C548 pad 1: GNDPWR -> -18V
- C548 pad 2: Net-(C544-Pad2) -> GNDPWR
- C549 pad 1: GNDPWR -> -18V
- C549 pad 2: Net-(C544-Pad2) -> GNDPWR
- C551 pad 1: GNDPWR -> Net-(C551-Pad1)
- C551 pad 2: -18V -> GNDPWR
- L44 pad 2: Net-(U45-EN) -> Net-(C468-Pad1)
- L461 pad 1: Net-(C464-Pad1) -> Net-(C468-Pad1)
- L461 pad 2: -2V5 -> /Low Voltage Power/Im2V5
- L55 pad 2: Net-(L55-Pad2) -> Net-(C551-Pad1)
- L56 pad 1: Net-(C544-Pad2) -> Net-(C551-Pad1)
- L56 pad 2: -18V -> /18V/im18
- R101 pad 1: /Offset Voltage Ladder/5V -> Net-(U11A--)
- R309 pad 1: Net-(U32B--) -> GND
- R309 pad 2: GND -> Net-(U32B--)
- R329 pad 1: Net-(U33A--) -> GND
- R329 pad 2: GND -> Net-(U33A--)
- R349 pad 1: Net-(U37B--) -> GND
- R349 pad 2: GND -> Net-(U37B--)
- R369 pad 1: Net-(U38A--) -> GND
- R369 pad 2: GND -> Net-(U38A--)
- R462 pad 1: Net-(C464-Pad1) -> -2V5
- R524 pad 1: Net-(U52-EN) -> /18V/i18
- R541 pad 1: Net-(C544-Pad2) -> -18V
- TP54 pad 1: Net-(C544-Pad2) -> -18V
- U11 pad 1: /Offset Voltage Ladder/5V -> Net-(U11A--)
- U11 pad 2: /Offset Voltage Ladder/5V -> Net-(U11A--)
- U30 pad 28: /DAC2752-1B/IOUT2 -> Net-(U30B-IOUT2BF)
- U30 pad 37: /DAC2752-1B/ROFS -> /DAC2752-1B/RIN
- U30 pad 38: /DAC2752-1B/ROFS -> /DAC2752-1B/RIN
- U30 pad 39: /DAC2752-1B/RFB -> /DAC2752-1B/Force
- U30 pad 46: /DAC2752-1A/RFB -> /DAC2752-1A/Force
- U30 pad 47: /DAC2752-1A/ROFS -> /DAC2752-1A/RIN
- U30 pad 48: /DAC2752-1A/ROFS -> /DAC2752-1A/RIN
- U30 pad 9: /DAC2752-1A/IOUT2 -> Net-(U30A-IOUT2AF)
- U35 pad 28: /DAC2752-2B/IOUT2 -> Net-(U35B-IOUT2BF)
- U35 pad 37: /DAC2752-2B/ROFS -> /DAC2752-2B/RIN
- U35 pad 38: /DAC2752-2B/ROFS -> /DAC2752-2B/RIN
- U35 pad 39: /DAC2752-2B/RFB -> /DAC2752-2B/Force
- U35 pad 46: /DAC2752-2A/RFB -> /DAC2752-2A/Force
- U35 pad 47: /DAC2752-2A/ROFS -> /DAC2752-2A/RIN
- U35 pad 48: /DAC2752-2A/ROFS -> /DAC2752-2A/RIN
- U35 pad 9: /DAC2752-2A/IOUT2 -> Net-(U35A-IOUT2AF)
- U45 pad 1: Net-(C464-Pad1) -> -2V5
- U45 pad 13: Net-(U45-EN) -> /Low Voltage Power/Im2V5
- U45 pad 15: Net-(U45-EN) -> /Low Voltage Power/Im2V5
- U45 pad 16: Net-(U45-EN) -> /Low Voltage Power/Im2V5
- U45 pad 20: Net-(C464-Pad1) -> -2V5
- U52 pad 13: Net-(U52-EN) -> /18V/i18
- U52 pad 15: Net-(U52-EN) -> /18V/i18
- U52 pad 16: Net-(U52-EN) -> /18V/i18
- U53 pad 1: Net-(C544-Pad2) -> -18V
- U53 pad 13: Net-(U53-EN) -> /18V/im18
- U53 pad 15: Net-(U53-EN) -> /18V/im18
- U53 pad 16: Net-(U53-EN) -> /18V/im18
- U53 pad 20: Net-(C544-Pad2) -> -18V
- U7 pad 22: /Monitor ADC/BufR+ -> unconnected-(U7-AIN1-Pad22)
- U7 pad 23: /Monitor ADC/BufR- -> unconnected-(U7-AIN2-Pad23)
- U81 pad 4: unconnected-(U81-QE-Pad4) -> /SHSel
- U81 pad 5: unconnected-(U81-QF-Pad5) -> /OffsetA2
- U81 pad 6: unconnected-(U81-QG-Pad6) -> /OffsetA1
- U81 pad 7: unconnected-(U81-QH-Pad7) -> /OffsetA0
- U85 pad 10: /Comp2A -> /Auxilary/DAC6
- U85 pad 11: /Comp2B -> /Auxilary/DAC7
- U85 pad 2: /DAC_SH1 -> /MonTC
- U85 pad 3: /DAC_SH2 -> /Ref2V16
- U85 pad 4: /MonTC -> /Auxilary/DAC2
- U85 pad 5: /Ref2V16 -> /Auxilary/DAC3
- U85 pad 8: /Comp1A -> /Auxilary/DAC4
- U85 pad 9: /Comp1B -> /Auxilary/DAC5
Routing:
- net /Comp1B: track 31.7 -> 0.00 mm, vias 2 -> 0
- net Net-(D52-A): track 0.00 -> 21.5 mm, vias 1 -> 0
- net /Comp2A: track 16.3 -> 0.00 mm, vias 1 -> 0
- net /Comp1A: track 13.4 -> 0.00 mm, vias 1 -> 0
- net Net-(U35A-IOUT2AF): track 0.00 -> 12.6 mm, vias 0 -> 2
- net Net-(U30A-IOUT2AF): track 0.00 -> 12.5 mm, vias 0 -> 2
- net /18V/im18: track 0.00 -> 12.1 mm
- net /18V/i18: track 0.00 -> 11.8 mm
- net Net-(U45-EN): track 10.9 -> 0.00 mm
- net /Low Voltage Power/Im2V5: track 0.00 -> 10.9 mm
- net Net-(U35A-IOUT2AS): track 2.46 -> 12.7 mm, vias 0 -> 2
- net Net-(U30A-IOUT2AS): track 2.51 -> 12.4 mm, vias 0 -> 2
- net -18V: track 177.7 -> 187.3 mm
- net GNDPWR: track 215.9 -> 225.3 mm, vias 159 -> 168
- net Net-(U35B-IOUT2BF): track 0.00 -> 8.79 mm
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
Commit message: S&H restored.  Now to touch up connections etc.
Parts:
- added C201: 10u, Parts:C_Rect_L31.5mm_W15.0mm_P27.50mm_MKS4, F.Cu at (209.3, 119.8)
- added C202: 0n1, Capacitor_SMD:C_0402_1005Metric, F.Cu at (200.8, 114.0)
- added C203: 10n, Capacitor_SMD:C_0603_1608Metric, F.Cu at (200.8, 116.5)
- added C204: 0n1, Capacitor_SMD:C_0402_1005Metric, F.Cu at (180.8, 126.8)
- added C205: 0n1, Capacitor_SMD:C_0402_1005Metric, F.Cu at (200.8, 119.0)
- added C206: 0u1, Capacitor_SMD:C_0402_1005Metric, F.Cu at (237.7, 116.7)
- added C207: 0u1, Capacitor_SMD:C_0402_1005Metric, F.Cu at (237.7, 118.7)
- added C208: 0u1, Capacitor_SMD:C_0402_1005Metric, F.Cu at (183.1, 144.7)
- added C209: 0u1, Capacitor_SMD:C_0402_1005Metric, F.Cu at (182.6, 149.2)
- added C210: 0u1, Capacitor_SMD:C_0402_1005Metric, F.Cu at (232.8, 126.2)
- added C211: 0u1, Capacitor_SMD:C_0402_1005Metric, F.Cu at (232.8, 128.2)
- added C212: 1u, Capacitor_SMD:C_0402_1005Metric, F.Cu at (200.8, 121.5)
- added C251: 10u, Parts:C_Rect_L31.5mm_W15.0mm_P27.50mm_MKS4, F.Cu at (209.3, 183.2)
- added C252: 0n1, Capacitor_SMD:C_0402_1005Metric, F.Cu at (193.2, 163.6)
- added C253: 10n, Capacitor_SMD:C_0603_1608Metric, F.Cu at (208.3, 160.8)
- added C254: 0n1, Capacitor_SMD:C_0402_1005Metric, F.Cu at (182.6, 189.6)
- added C255: 0n1, Capacitor_SMD:C_0402_1005Metric, F.Cu at (230.0, 176.6)
- added C256: 0u1, Capacitor_SMD:C_0402_1005Metric, F.Cu at (232.7, 177.2)
- added C257: 0u1, Capacitor_SMD:C_0402_1005Metric, F.Cu at (229.1, 181.3)
- added C258: 0u1, Capacitor_SMD:C_0402_1005Metric, F.Cu at (195.3, 169.4)
- added C259: 0u1, Capacitor_SMD:C_0402_1005Metric, F.Cu at (188.7, 165.8)
- added C260: 0u1, Capacitor_SMD:C_0402_1005Metric, F.Cu at (244.8, 167.7)
- added C261: 0u1, Capacitor_SMD:C_0402_1005Metric, F.Cu at (244.8, 169.7)
- added C262: 1u, Capacitor_SMD:C_0402_1005Metric, F.Cu at (212.2, 159.4)
- added D21: SM4007PL, Parts:D_SOD-123FL, F.Cu at (226.2, 143.9)
- added D22: SM4007PL, Parts:D_SOD-123FL, F.Cu at (226.2, 147.3)
- added D23: SM4007PL, Parts:D_SOD-123FL, F.Cu at (226.2, 150.7)
- added D26: SM4007PL, Parts:D_SOD-123FL, F.Cu at (219.8, 161.1)
- added D27: SM4007PL, Parts:D_SOD-123FL, F.Cu at (225.1, 162.2)
- added D28: SM4007PL, Parts:D_SOD-123FL, F.Cu at (214.7, 162.2)
- added JP21: SolderJumper_2_Open, Parts:JumperOpen, F.Cu at (179.4, 122.5)
- added JP22: SolderJumper_2_Open, Parts:JumperOpen, F.Cu at (188.2, 186.2)
- added K21: G6K-2FY, 5V, Relay_SMD:Relay_DPDT_Omron_G6K-2G-Y, F.Cu at (219.8, 138.2)
- added K22: G6K-2FY, 5V, Relay_SMD:Relay_DPDT_Omron_G6K-2G-Y, F.Cu at (219.8, 167.4)
- added L21: 600, Inductor_SMD:L_0603_1608Metric, F.Cu at (200.8, 124.0)
- added L25: 600, Inductor_SMD:L_0603_1608Metric, F.Cu at (212.2, 156.4)
- added Q201: AO3400A, Parts:SOT-23, F.Cu at (226.7, 134.4)
- added Q202: AO3401A, Parts:SOT-23, F.Cu at (231.3, 139.3)
- added Q203: AO3400A, Parts:SOT-23, F.Cu at (226.8, 139.8)
- added Q204: AO3400A, Parts:SOT-23, F.Cu at (186.1, 112.0)
- added Q205: AO3400A, Parts:SOT-23, F.Cu at (186.1, 117.3)
- added Q206: AO3400A, Parts:SOT-23, F.Cu at (186.1, 121.8)
- added Q207: AO3400A, Parts:SOT-23, F.Cu at (186.1, 126.2)
- added Q251: AO3400A, Parts:SOT-23, F.Cu at (225.1, 157.9)
- added Q252: AO3401A, Parts:SOT-23, F.Cu at (214.7, 157.9)
- added Q253: AO3400A, Parts:SOT-23, F.Cu at (219.9, 157.9)
- added Q254: AO3400A, Parts:SOT-23, F.Cu at (203.6, 168.8)
- added Q255: AO3400A, Parts:SOT-23, F.Cu at (203.4, 164.8)
- added Q256: AO3400A, Parts:SOT-23, F.Cu at (188.7, 189.6)
- added Q257: AO3400A, Parts:SOT-23, F.Cu at (185.2, 189.6)
- added R201: 16k, Resistor_SMD:R_0603_1608Metric, F.Cu at (200.8, 126.5)
- added R202: 100k, Resistor_SMD:R_0402_1005Metric, F.Cu at (206.1, 114.8)
- added R203: 1k, Resistor_SMD:R_0805_2012Metric, F.Cu at (200.3, 139.6)
- added R204: 1k, Resistor_SMD:R_0805_2012Metric, F.Cu at (203.2, 139.6)
- added R205: 1k, Resistor_SMD:R_0805_2012Metric, F.Cu at (206.2, 139.6)
- added R206: 1k, Resistor_SMD:R_0805_2012Metric, F.Cu at (209.2, 139.6)
- added R207: 10k, Resistor_SMD:R_0402_1005Metric, F.Cu at (206.1, 116.8)
- added R208: 10k, Resistor_SMD:R_0402_1005Metric, F.Cu at (206.1, 118.8)
- added R209: 100k, Resistor_SMD:R_0402_1005Metric, F.Cu at (206.1, 120.8)
- added R210: 10, Resistor_SMD:R_0402_1005Metric, F.Cu at (206.1, 122.7)
- added R211: 330, Resistor_SMD:R_0402_1005Metric, F.Cu at (206.1, 124.7)
- added R212: 1k, Resistor_SMD:R_0402_1005Metric, F.Cu at (206.1, 126.7)
- added R213: 8k2, Resistor_SMD:R_0603_1608Metric, F.Cu at (200.8, 129.1)
- added R214: 200, Resistor_SMD:R_0402_1005Metric, F.Cu at (182.8, 147.2)
- added R251: 16k, Resistor_SMD:R_0603_1608Metric, F.Cu at (192.7, 161.6)
- added R252: 100k, Resistor_SMD:R_0402_1005Metric, F.Cu at (195.1, 159.8)
- added R253: 1k, Resistor_SMD:R_0805_2012Metric, F.Cu at (209.2, 156.7)
- added R254: 1k, Resistor_SMD:R_0805_2012Metric, F.Cu at (206.2, 156.7)
- added R255: 1k, Resistor_SMD:R_0805_2012Metric, F.Cu at (203.2, 156.7)
- added R256: 1k, Resistor_SMD:R_0805_2012Metric, F.Cu at (200.3, 156.7)
- added R257: 10k, Resistor_SMD:R_0402_1005Metric, F.Cu at (213.8, 171.7)
- added R258: 10k, Resistor_SMD:R_0402_1005Metric, F.Cu at (214.7, 155.7)
- added R259: 100k, Resistor_SMD:R_0402_1005Metric, F.Cu at (225.1, 155.7)
- added R260: 10, Resistor_SMD:R_0402_1005Metric, F.Cu at (232.6, 175.8)
- added R261: 330, Resistor_SMD:R_0402_1005Metric, F.Cu at (228.0, 176.1)
- added R262: 1k, Resistor_SMD:R_0402_1005Metric, F.Cu at (185.8, 176.8)
- added R263: 8k2, Resistor_SMD:R_0603_1608Metric, F.Cu at (191.8, 172.2)
- added R265: 200, Resistor_SMD:R_0402_1005Metric, F.Cu at (181.8, 174.1)
- added RN21: 100R × 4, Resistor_SMD:R_Array_Convex_4x0603, F.Cu at (179.2, 114.5)
- added RN22: 100R × 4, Resistor_SMD:R_Array_Convex_4x0603, F.Cu at (185.2, 173.4)
- added U19: TCA0372, Package_SO:SOIC-16W_7.5x10.3mm_P1.27mm, F.Cu at (204.8, 148.2)
- added U21: OPA828DGN, Parts:VSSOP-8-1EP_3x3mm_P0.65mm_EP1.57x1.89mm, F.Cu at (232.6, 117.8)
- added U22: OPA2197D, Parts:OPA2197, F.Cu at (188.8, 148.2)
- added U23: DG419D, Package_SO:SOIC-8_3.9x4.9mm_P1.27mm, F.Cu at (239.1, 127.3)
- added U25: OPA828DGN, Parts:VSSOP-8-1EP_3x3mm_P0.65mm_EP1.57x1.89mm, F.Cu at (230.0, 179.1)
- added U26: OPA2197D, Parts:OPA2197, F.Cu at (191.8, 167.8)
- added U27: DG419D, Package_SO:SOIC-8_3.9x4.9mm_P1.27mm, F.Cu at (239.2, 169.1)
- moved C101 153.1 mm to (134.7, 79.8)
- moved C102 153.1 mm to (142.1, 79.8)
- moved C104 153.1 mm to (134.1, 84.7)
- moved C105 153.1 mm to (138.4, 75.7)
- moved R101 153.1 mm to (131.4, 75.6)
- moved R102 153.1 mm to (131.4, 77.1)
- moved R103 153.1 mm to (131.4, 78.6)
- moved R104 153.1 mm to (131.4, 80.1)
- moved R105 153.1 mm to (131.4, 81.6)
- moved R106 153.1 mm to (131.4, 83.1)
- moved R107 153.1 mm to (131.4, 84.6)
- moved R108 153.1 mm to (145.4, 78.6)
- moved R109 153.1 mm to (145.4, 80.1)
- moved R110 153.1 mm to (145.4, 81.6)
- moved R111 153.1 mm to (145.4, 83.1)
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Routing:
- net Net-(U27-S1): track 0.00 -> 58.2 mm, vias 0 -> 8
- net /Sample Hold 2/Drive: track 0.00 -> 33.9 mm
- net GND: track 57.8 -> 75.8 mm
- net /Sample Hold 2/SH: track 0.00 -> 17.0 mm
- net Net-(U19B--): track 0.00 -> 15.2 mm
- net Net-(U19A--): track 0.00 -> 14.6 mm
- net /Sample Hold 2/SHGnd: track 0.00 -> 9.78 mm
- net /Sample Hold 1/Drive: track 0.00 -> 8.80 mm
- net /Sample Hold 2/Sample: track 0.00 -> 8.15 mm
- net Net-(C255-Pad1): track 0.00 -> 7.20 mm
- net GNDPWR: track 225.3 -> 232.0 mm, vias 168 -> 171
- net Net-(Q252-G): track 0.00 -> 6.65 mm
- net Net-(D26-A): track 0.00 -> 5.92 mm
- net Net-(D26-K): track 0.00 -> 5.92 mm
- net Net-(K22-Pad2): track 0.00 -> 5.70 mm
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Other:
- board size 250 x 150 mm -> 263.3 x 157.7 mm
