File: cpu.kicad_sch (KiCad schematic)
At the start: 1 part

Commit message: Schematic complete, maybe
Parts:
- removed U?: ESP32-C6-MINI-1, RF_Module:ESP32-C6-MINI-1, symbol RF_Module:ESP32-C6-MINI-1
- added C80, C82, C86: 10u, Capacitor_SMD:C_0603_1608Metric, symbol Device:C
- added C81, C84: 1u, Capacitor_SMD:C_0402_1005Metric, symbol Device:C
- added C83, C85, C87, C88, C89: 0u1, Capacitor_SMD:C_0402_1005Metric, symbol Device:C
- added J81: Conn_01x03_Pin, symbol Connector:Conn_01x03_Pin
- added J82, J83: Conn_Coaxial, symbol Connector:Conn_Coaxial
- added J84: Conn_01x02_Pin, symbol Connector:Conn_01x02_Pin
- added L81: 100, Inductor_SMD:L_0603_1608Metric, symbol Parts:L_Ferrite_Power
- added L82: 600, Inductor_SMD:L_0603_1608Metric, symbol Parts:L_Ferrite_Power
- added R81, R86, R87: 10k, Resistor_SMD:R_0402_1005Metric, symbol Device:R
- added R82: 1k, Resistor_SMD:R_0402_1005Metric, symbol Device:R
- added R83, R84, R85: 0, Resistor_SMD:R_0402_1005Metric, symbol Device:R
- added SW81, SW82: SW_Push, symbol Switch:SW_Push
- added U8: ESP32-C6-MINI-1U, RF_Module:ESP32-C6-MINI-1, symbol Parts:ESP32-C6-MINI-1U
- added U81, U82: 74HC595, Package_SO:SOIC-16_3.9x9.9mm_P1.27mm, symbol 74xx:74HC595
- added U83: ISOW7842, Package_SO:SOIC-16W_7.5x10.3mm_P1.27mm, symbol Parts:ISOW7842
Connections:
- new net: C82.1, C83.1, L82.2, U83.1 (V_{CC})
- new net: C80.1, C81.1, L81.2, U8.3 (3V3)
- new net: R81.1, R82.2, SW81.1
- new net: U81.9 (QH'), U82.14 (SER)
- new net: C84.1, R82.1, U8.8 (EN)
- new net: J83.1 (In), U83.12 (INC)
- new net: R86.2, U8.22 (IO8)
- new net: J82.1 (In), U83.13 (OUTB)
- new net: J81.1 (Pin_1), U8.31 (TXD0)
- new net: J81.2 (Pin_2), U8.30 (RXD0)
- new net: J84.1 (Pin_1), SW82.1, U8.23 (IO9)
- new net: C85.1, C86.1, U83.16 (V_{ISO})
- new net +3V3: L81.1, L82.1, R81.2, R86.1
- new net +3V3A: C88.1, C89.1, R87.2, U81.16 (VCC), U82.16 (VCC)
- new net Earth: J82.2 (Ext), J83.2 (Ext), U83.10 (SEL), U83.11 (IND), U83.15 (GND2), U83.9 (GND2)
- new net GND1: C80.2, C81.2, C82.2, C83.2, C84.2, C85.2, C86.2, C87.2, C88.2, C89.2, J81.3 (Pin_3), J84.2 (Pin_2), SW81.2, SW82.2, U8.1 (GND), U8.11 (GND), U8.14 (GND), U8.2 (GND), U8.36 (GND), U8.37 (GND), U8.38 (GND), U8.39 (GND), U8.40 (GND), U8.41 (GND), U8.42 (GND), U8.43 (GND), U8.44 (GND), U8.45 (GND), U8.46 (GND), U8.47 (GND), U8.48 (GND), U8.49 (GND), U8.50 (GND), U8.51 (GND), U8.52 (GND), U8.53 (GND), U81.13 (~{OE}), U81.8 (GND), U82.13 (~{OE}), U82.8 (GND), U83.2 (GND1), U83.3 (INA), U83.8 (GND1)
- new net LATCH: U8.28 (IO22), U81.12 (RCLK), U82.12 (RCLK)
- new net MISO: U8.5 (IO2)
- new net MOSI: R85.1, U81.14 (SER)
- new net MonA0: U82.4 (QE)
- new net MonA1: U82.5 (QF)
- new net MonB0: U82.6 (QG)
- new net MonB1: U82.7 (QH)
- new net OffsetA0: U82.15 (QA)
- new net OffsetA1: U82.1 (QB)
- new net OffsetA2: U82.2 (QC)
- new net PWR_EN: U8.20 (IO15)
- new net SCK: R84.1, U81.11 (SRCLK), U82.11 (SRCLK)
- new net SHHoldG1: U81.3 (QD)
- new net SHHoldG2: U81.7 (QH)
- new net SHOutEn1: U81.15 (QA)
- new net SHOutEn2: U81.4 (QE)
- new net SHSample1: U81.1 (QB)
- new net SHSample2: U81.5 (QF)
- new net SHSampleG1: U81.2 (QC)
- new net SHSampleG2: U81.6 (QG)
- new net SHSel: U82.3 (QD)
- new net TCK: R84.2, U8.15 (IO6)
- new net TDI: R83.2, U8.10 (IO5)
- new net TDO: R85.2, U8.16 (IO7)
- new net TMS: U8.9 (IO4)
- new net TRIGIN: R83.1, U83.4 (INB)
- new net TRIGOUT: U8.6 (IO3), U83.5 (OUTC)
- new net USB_D+: U8.19 (IO14)
- new net USB_D-: U8.18 (IO13)
- new net ~{CS2}: U8.24 (IO18)
- new net ~{CS3}: U8.25 (IO19)
- new net ~{CS4}: U8.26 (IO20)
- new net ~{CS5}: U8.27 (IO21)
- new net ~{LDAC}: U8.29 (IO23)
- new net ~{SRCLR}: C87.1, R87.1, U81.10 (~{SRCLR}), U82.10 (~{SRCLR})
- no-connect marks 0 -> 3

Commit message: Part selection
Parts:
- removed R83, R84, R85: 0, Resistor_SMD:R_0402_1005Metric, symbol Device:R
- J81, J82, J83, J84: now left out of the parts list
- R81, R86, R87: LCSC (none) -> C25744
- R82: LCSC (none) -> C11702
Connections:
- net TCK is gone; now on net SCK: U8.15 (IO6)
- net TDI is gone; now on net TRIGIN: U8.10 (IO5)
- net TDO is gone; now on net MOSI: U8.16 (IO7)
- net TMS: no longer names the net of U8.9 (IO4)
Other:
- moved on the sheet: R86

Commit message: ERC passes.
Parts:
- added R83: 33, Resistor_SMD:R_0603_1608Metric, symbol Device:R
- added R84: 100, Resistor_SMD:R_0402_1005Metric, symbol Device:R
- J82, J83: footprint (none) -> Connector_Coaxial:SMA_Amphenol_901-144_Vertical
- SW81, SW82: footprint (none) -> Button_Switch_SMD:SW_SPST_TS-1088-xR020; LCSC (none) -> C720477
Connections:
- net at J83.1 (In): now also R84.2; no longer U83.12 (INC)
- net at J82.1 (In): now also R83.2; no longer U83.13 (OUTB)
- net GND1 renamed GNDPWR
- new net: R83.1, U83.13 (OUTB)
- new net: R84.1, U83.12 (INC)
- no-connect marks 3 -> 7
Other:
- moved on the sheet: J82, J83

Commit message: Everything assigned except for wierd shit.
Parts:
- added C90: 0u1, Capacitor_SMD:C_0402_1005Metric, symbol Device:C
- added U83: 74HC595, Package_SO:SOIC-16_3.9x9.9mm_P1.27mm, symbol 74xx:74HC595
- renumbered U83 to U84
Connections:
- net +3V3A: now also C90.1, U83.16 (VCC)
- net GNDPWR: now also C90.2, U83.13 (~{OE}), U83.8 (GND)
- net LATCH: now also U83.12 (RCLK)
- net SCK: now also U83.11 (SRCLK)
- net ~{SRCLR}: now also U83.10 (~{SRCLR})
- net at U82.9 (QH'): now also U83.14 (SER)
- new net Sel1A: U83.15 (QA)
- new net Sel1B: U83.1 (QB)
- new net Sel2A: U83.2 (QC)
- new net Sel2B: U83.3 (QD)
- no-connect marks 7 -> 11
Other:
- moved on the sheet: C87, C88, C89, R87, U81, U82

Commit message: Layout underway
Parts:
- J81: footprint (none) -> Parts:PinHeader_1x03_P2.54mm_Vertical
- J84: footprint (none) -> Parts:PinHeader_1x02_P2.54mm_Vertical
Changed lines of the file:
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@@
 			)
 		)
-		(property "Footprint" ""
+		(property "Footprint" "Parts:PinHeader_1x03_P2.54mm_Vertical"
 			(at 123.19 50.8 0)
 			(effects
@@
 			)
 		)
-		(property "Footprint" ""
+		(property "Footprint" "Parts:PinHeader_1x02_P2.54mm_Vertical"
 			(at 76.2 88.9 0)
 			(effects

Commit message: Tweaks following spice simulation.
Parts:
- C83: value 0u1 -> 1u; LCSC C307331 -> C52923
Connections:
- net MonA0: now also U82.3 (QD); no longer U82.4 (QE)
- net MonA1: now also U82.2 (QC); no longer U82.5 (QF)
- net MonB0: now also U82.1 (QB); no longer U82.6 (QG)
- net MonB1: now also U82.15 (QA); no longer U82.7 (QH)
- net OffsetA0: now also U82.7 (QH); no longer U82.15 (QA)
- net OffsetA1: now also U82.6 (QG); no longer U82.1 (QB)
- net OffsetA2: now also U82.5 (QF); no longer U82.2 (QC)
- net SHHoldG1: now also U81.4 (QE); no longer U81.3 (QD)
- net SHHoldG2: now also U81.15 (QA); no longer U81.7 (QH)
- net SHOutEn1: now also U81.7 (QH); no longer U81.15 (QA)
- net SHOutEn2: now also U81.3 (QD); no longer U81.4 (QE)
- net SHSample1: now also U81.6 (QG); no longer U81.1 (QB)
- net SHSample2: now also U81.2 (QC); no longer U81.5 (QF)
- net SHSampleG1: now also U81.5 (QF); no longer U81.2 (QC)
- net SHSampleG2: now also U81.1 (QB); no longer U81.6 (QG)
- net SHSel: now also U82.4 (QE); no longer U82.3 (QD)
- net Sel1A: now also U83.7 (QH); no longer U83.15 (QA)
- net Sel1B: now also U83.6 (QG); no longer U83.1 (QB)
- net Sel2A: now also U83.5 (QF); no longer U83.2 (QC)
- net Sel2B: now also U83.4 (QE); no longer U83.3 (QD)
Changed lines of the file:
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@@
 	)
 	(no_connect
-		(at 194.31 118.11)
+		(at 193.04 107.95)
 	)
 	(no_connect
@@
 	)
 	(no_connect
-		(at 80.01 53.34)
+		(at 193.04 113.03)
 	)
 	(no_connect
-		(at 193.04 128.27)
+		(at 80.01 53.34)
 	)
 	(no_connect
-		(at 194.31 123.19)
+		(at 193.04 105.41)
 	)
 	(no_connect
-		(at 167.64 59.69)
+		(at 193.04 128.27)
 	)
 	(no_connect
-		(at 194.31 120.65)
+		(at 193.04 110.49)
 	)
 	(no_connect
-		(at 80.01 63.5)
+		(at 167.64 59.69)
 	)
 	(no_connect
-		(at 194.31 115.57)
+		(at 80.01 63.5)
 	)
 	(no_connect
@@
 	(wire
 		(pts
-			(xy 193.04 107.95) (xy 194.31 107.95)
+			(xy 193.04 120.65) (xy 194.31 120.65)
 		)
 		(stroke
@@
 	(wire
 		(pts
-			(xy 193.04 115.57) (xy 194.31 115.57)
-		)
-		(stroke
-			(width 0)
-			(type default)
-		)
-	)
-	(wire
-		(pts
 			(xy 63.5 66.04) (xy 80.01 66.04)
 		)
@@
 	(wire
 		(pts
-			(xy 193.04 118.11) (xy 194.31 118.11)
-		)
-		(stroke
-			(width 0)
-			(type default)
-		)
-	)
-	(wire
-		(pts
 			(xy 116.84 118.11) (xy 124.46 118.11)
 		)
@@
 	(wire
 		(pts
-			(xy 193.04 113.03) (xy 194.31 113.03)
+			(xy 193.04 115.57) (xy 194.31 115.57)
 		)
 		(stroke
@@
 	(wire
 		(pts
-			(xy 193.04 105.41) (xy 194.31 105.41)
+			(xy 193.04 123.19) (xy 194.31 123.19)
 		)
 		(stroke
@@
 	(wire
 		(pts
-			(xy 193.04 120.65) (xy 194.31 120.65)
-		)
-		(stroke
-			(width 0)
-			(type default)
-		)
-	)
-	(wire
-		(pts
 			(xy 57.15 46.99) (xy 57.15 48.26)
 		)
@@
 	(wire
 		(pts
-			(xy 193.04 110.49) (xy 194.31 110.49)
+			(xy 193.04 118.11) (xy 194.31 118.11)
 		)
 		(stroke
@@
 	(wire
 		(pts
-			(xy 193.04 123.19) (xy 194.31 123.19)
-		)
-		(stroke
-			(width 0)
-			(type default)
-		)
-	)
-	(wire
-		(pts
 			(xy 160.02 128.27) (xy 160.02 105.41)
 		)
@@
 				)
 				(justify left)
-				(hide yes)
 			)
 		)
@@
 				)
 				(justify left)
-				(hide yes)
 			)
 		)
@@
 				)
 				(justify left)
-				(hide yes)
 			)
 		)
@@
 	(hierarchical_label "SHSample1"
 		(shape output)
-		(at 91.44 107.95 0)
+		(at 91.44 120.65 0)
 		(effects
 			(font
@@
 	(hierarchical_label "SHHoldG1"
 		(shape output)
-		(at 91.44 113.03 0)
+		(at 91.44 115.57 0)
 		(effects
 			(font
@@
 	(hierarchical_label "SHSampleG2"
 		(shape output)
-		(at 91.44 120.65 0)
+		(at 91.44 107.95 0)
 		(effects
 			(font
@@
 	(hierarchical_label "OffsetA0"
 		(shape output)
-		(at 146.05 105.41 0)
+		(at 146.05 123.19 0)
 		(effects
 			(font
@@
 	(hierarchical_label "MonA1"
 		(shape output)
-		(at 146.05 118.11 0)
+		(at 146.05 110.49 0)
 		(effects
 			(font
@@
 	(hierarchical_label "Sel2B"
 		(shape output)
-		(at 194.31 113.03 0)
+		(at 194.31 115.57 0)
 		(effects
 			(font
@@
 	(hierarchical_label "SHHoldG2"
 		(shape output)
-		(at 91.44 123.19 0)
+		(at 91.44 105.41 0)
 		(effects
 			(font
@@
 	(hierarchical_label "SHOutEn2"
 		(shape output)
-		(at 91.44 115.57 0)
+		(at 91.44 113.03 0)
 		(effects
 			(font
@@
 	(hierarchical_label "Sel1B"
 		(shape output)
-		(at 194.31 107.95 0)
+		(at 194.31 120.65 0)
 		(effects
 			(font
@@
 	(hierarchical_label "SHSel"
 		(shape output)
-		(at 146.05 113.03 0)
+		(at 146.05 115.57 0)
 		(effects
 			(font
@@
 	(hierarchical_label "SHOutEn1"
 		(shape output)
-		(at 91.44 105.41 0)
+		(at 91.44 123.19 0)
 		(effects
 			(font
@@
 	(hierarchical_label "OffsetA2"
 		(shape output)
-		(at 146.05 110.49 0)
+		(at 146.05 118.11 0)
 		(effects
 			(font
@@
 	(hierarchical_label "MonB1"
 		(shape output)
-		(at 146.05 123.19 0)
+		(at 146.05 105.41 0)
 		(effects
 			(font
@@
 	(hierarchical_label "SHSampleG1"
 		(shape output)
-		(at 91.44 110.49 0)
+		(at 91.44 118.11 0)
 		(effects
 			(font
@@
 	(hierarchical_label "MonB0"
 		(shape output)
-		(at 146.05 120.65 0)
+		(at 146.05 107.95 0)
 		(effects
 			(font
@@
 	(hierarchical_label "Sel1A"
 		(shape output)
-		(at 194.31 105.41 0)
+		(at 194.31 123.19 0)
 		(effects
 			(font
@@
 	(hierarchical_label "Sel2A"
 		(shape output)
-		(at 194.31 110.49 0)
+		(at 194.31 118.11 0)
 		(effects
 			(font
@@
 	(hierarchical_label "MonA0"
 		(shape output)
-		(at 146.05 115.57 0)
+		(at 146.05 113.03 0)
 		(effects
 			(font
@@
 	(hierarchical_label "SHSample2"
 		(shape output)
-		(at 91.44 118.11 0)
+		(at 91.44 110.49 0)
 		(effects
 			(font
@@
 	(hierarchical_label "OffsetA1"
 		(shape output)
-		(at 146.05 107.95 0)
+		(at 146.05 120.65 0)
 		(effects
 			(font
@@
 			)
 		)
-		(property "Value" "0u1"
+		(property "Value" "1u"
 			(at 142.24 48.768 0)
 			(effects
@@
 			)
 		)
-		(property "Datasheet" "50V"
+		(property "Datasheet" "25V"
 			(at 142.24 50.8 0)
 			(effects
@@
 			)
 		)
-		(property "LCSC" "C307331"
+		(property "LCSC" "C52923"
 			(at 142.24 50.8 0)
 			(effects
@@
 		(dnp no)
 		(property "Reference" "C82"
-			(at 136.906 48.768 0)
+			(at 137.16 45.72 0)
 			(effects
 				(font
 					(size 1.27 1.27)
 				)
-				(justify right)
 			)
 		)
@@
 			)
 		)
-		(property "Datasheet" "~"
+		(property "Datasheet" "200mA / 450mΩ"
 			(at 151.13 46.99 0)
 			(effects
@@
 			)
 		)
-		(property "Datasheet" "2A / 50mOhm"
+		(property "Datasheet" "2A / 50mΩ"
 			(at 88.9 31.75 0)
 			(effects

Commit message: About to delete scan...
Parts:
- U84: Stock (none) -> 2
Connections:
- net MonA0: now also U83.3 (QD); no longer U82.3 (QD)
- net MonA1: now also U83.2 (QC); no longer U82.2 (QC)
- net MonB0: now also U83.1 (QB); no longer U82.1 (QB)
- net MonB1: now also U83.15 (QA); no longer U82.15 (QA)
