File: fda.kicad_sch (KiCad schematic)
At the start: 42 parts, among them U706 OPA2197D, U73 OPA2388DGK, U74 THS4551IDGK

Commit message: About to delete scan...
Parts:
- C720, C721: LCSC (none) -> C307500; now in the parts list
- R720, R721: footprint Capacitor_SMD:C_0402_1005Metric -> Resistor_SMD:R_0402_1005Metric
- R722, R723: footprint Capacitor_SMD:C_0603_1608Metric -> Resistor_SMD:R_0402_1005Metric; LCSC C22765 -> C11702
- U706: Stock (none) -> 30
- U73: Stock (none) -> 14
- U74: value THS4551IDGK -> THS4521IDGK; Stock (none) -> 3
Connections:
- net IN+: now also RN72.6; no longer RN72.7
- net IN-: now also RN73.7; no longer RN73.6
- net Out+: now also RN73.6; no longer RN73.7
- net Out-: now also RN72.7; no longer RN72.6
- net S2Bias: now reaches C725.1, R721.2, R728.1, R729.1
Other:
- moved on the sheet: R732, R735
