File: common2752.kicad_sch (KiCad schematic)
At the start: 8 parts, among them U1 OPA2189D, U30 LTC2752B, U35 LTC2752B, U36 OPA2189D

Commit message: Schematic complete, maybe
Parts:
- added C385, C386: 10u, Capacitor_SMD:C_0603_1608Metric, symbol Device:C
- added L31, L32: 600, Inductor_SMD:L_0603_1608Metric, symbol Parts:L_Ferrite_Power
- C381, C383: footprint (none) -> Capacitor_SMD:C_0402_1005Metric; LCSC (none) -> C307331
- C382, C384: value 10n -> 0u1; footprint (none) -> Capacitor_SMD:C_0402_1005Metric; LCSC (none) -> C307331
- U31: renamed from U1; LCSC (none) -> C881489; now left out of the parts list
- U36: LCSC (none) -> C881489; now left out of the parts list
Connections:
- net GND: now also C385.2, C386.2
- net +3V3 renamed 3V3-1
- net 3V3-1: now also C385.1, L31.2; no longer C383.1, U35.16 (VDD), U35.19 (~{CLR})
- new net +3V3A: L31.1, L32.1
- new net 3V3-2: C383.1, C386.1, L32.2, U35.16 (VDD), U35.19 (~{CLR})
Other:
- moved on the sheet: C381, C383

Commit message: ERC passes.
Parts:
- U31, U36: value OPA2189D -> OPA2189DGK; footprint Package_SO:SOIC-8_3.9x4.9mm_P1.27mm -> Package_SO:MSOP-8_3x3mm_P0.65mm; symbol Parts:OPA2189D -> Parts:OPA2189DGK
Connections:
- net GND renamed GNDPWR
- net GNDPWR: now also U30.10 (GND), U30.27 (GND), U30.30 (GND), U30.7 (GND), U35.10 (GND), U35.27 (GND), U35.30 (GND), U35.7 (GND)
Changed lines of the file:
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@@
 		(dnp no)
 		(property "Reference" "C384"
+			(at 119.38 115.57 0)
+			(effects
+				(font
+					(size 1.27 1.27)
+				)
+				(justify left top)
+			)
+		)
+		(property "Value" "0u1"
 			(at 119.38 113.03 0)
 			(effects
@@
 				)
 				(justify left bottom)
-			)
-		)
-		(property "Value" "0u1"
-			(at 119.38 115.57 0)
-			(effects
-				(font
-					(size 1.27 1.27)
-				)
-				(justify left top)
 			)
 		)
@@
 		)
 		(property "Value" "10u"
-			(at 43.18 77.216 0)
+			(at 43.18 73.152 0)
 			(effects
 				(font
@@
 		(dnp no)
 		(property "Reference" "C382"
+			(at 119.38 69.85 0)
+			(effects
+				(font
+					(size 1.27 1.27)
+				)
+				(justify left top)
+			)
+		)
+		(property "Value" "0u1"
 			(at 119.38 67.31 0)
 			(effects
@@
 				)
 				(justify left bottom)
-			)
-		)
-		(property "Value" "0u1"
-			(at 119.38 69.85 0)
-			(effects
-				(font
-					(size 1.27 1.27)
-				)
-				(justify left top)
 			)
 		)
@@
 	)
 	(symbol
-		(lib_id "Parts:OPA2189D")
+		(lib_id "Parts:OPA2189DGK")
 		(at 110.49 114.3 0)
 		(mirror y)
@@
 			)
 		)
-		(property "Value" "OPA2189D"
+		(property "Value" "OPA2189DGK"
 			(at 110.49 114.3 0)
 			(effects
@@
 			)
 		)
-		(property "Footprint" "Package_SO:SOIC-8_3.9x4.9mm_P1.27mm"
+		(property "Footprint" "Package_SO:MSOP-8_3x3mm_P0.65mm"
 			(at 111.76 114.3 0)
 			(effects
@@
 	)
 	(symbol
-		(lib_id "Parts:OPA2189D")
+		(lib_id "Parts:OPA2189DGK")
 		(at 110.49 68.58 0)
 		(mirror y)
@@
 			)
 		)
-		(property "Value" "OPA2189D"
+		(property "Value" "OPA2189DGK"
 			(at 110.49 68.58 0)
 			(effects
@@
 			)
 		)
-		(property "Footprint" "Package_SO:SOIC-8_3.9x4.9mm_P1.27mm"
+		(property "Footprint" "Package_SO:MSOP-8_3x3mm_P0.65mm"
 			(at 111.76 68.58 0)
 			(effects
@@
 		(dnp no)
 		(property "Reference" "C381"
+			(at 49.53 76.962 0)
+			(effects
+				(font
+					(size 1.27 1.27)
+				)
+				(justify right)
+			)
+		)
+		(property "Value" "0u1"
 			(at 49.53 73.152 0)
-			(effects
-				(font
-					(size 1.27 1.27)
-				)
-				(justify left)
-			)
-		)
-		(property "Value" "0u1"
-			(at 49.53 76.962 0)
 			(effects
 				(font
@@
 		)
 		(property "Value" "10u"
-			(at 43.18 122.936 0)
+			(at 43.18 118.872 0)
 			(effects
 				(font
@@
 		(dnp no)
 		(property "Reference" "C383"
+			(at 49.53 122.682 0)
+			(effects
+				(font
+					(size 1.27 1.27)
+				)
+				(justify right)
+			)
+		)
+		(property "Value" "0u1"
 			(at 49.53 118.872 0)
 			(effects
 				(font
-					(size 1.27 1.27)
-				)
-				(justify left)
-			)
-		)
-		(property "Value" "0u1"
-			(at 49.53 122.682 0)
-			(effects
-				(font

Commit message: Everything assigned except for wierd shit.
Parts:
- U30, U35: LCSC (none) -> C682625
Changed lines of the file:
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@@
+			)
+		)
+		(property "LCSC" "C682625"
+			(at 66.04 66.04 0)
+			(effects
+				(font
+					(size 1.27 1.27)
+				)
+				(hide yes)
 			)
 		)
@@
 			(effects
 				(font
+					(size 1.27 1.27)
+				)
+				(hide yes)
+			)
+		)
+		(property "LCSC" "C682625"
+			(at 66.04 111.76 0)
+			(effects
+				(font

Commit message: Whew.  DACs routed
Parts:
- U30, U35: footprint Package_QFP:LQFP-48_7x7mm_P0.5mm -> Parts:LQFP-48_7x7mm_P0.5mm
- U31, U36: footprint Package_SO:MSOP-8_3x3mm_P0.65mm -> Parts:OPA2189
Changed lines of the file:
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@@
 			)
 		)
-		(property "Footprint" "Package_QFP:LQFP-48_7x7mm_P0.5mm"
+		(property "Footprint" "Parts:LQFP-48_7x7mm_P0.5mm"
 			(at 66.04 58.42 0)
 			(effects
@@
 			)
 		)
-		(property "Footprint" "Package_QFP:LQFP-48_7x7mm_P0.5mm"
+		(property "Footprint" "Parts:LQFP-48_7x7mm_P0.5mm"
 			(at 66.04 104.14 0)
 			(effects
@@
 			)
 		)
-		(property "Footprint" "Package_SO:MSOP-8_3x3mm_P0.65mm"
+		(property "Footprint" "Parts:OPA2189"
 			(at 111.76 114.3 0)
 			(effects
@@
 			)
 		)
-		(property "Footprint" "Package_SO:MSOP-8_3x3mm_P0.65mm"
+		(property "Footprint" "Parts:OPA2189"
 			(at 111.76 68.58 0)
 			(effects

Commit message: Tweaks following spice simulation.
Parts:
- C381, C383: value 0u1 -> 1u; LCSC C307331 -> C52923
Changed lines of the file:
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@@
 			)
 		)
-		(property "Datasheet" "~"
+		(property "Datasheet" "200mA / 450mΩ"
 			(at 39.37 116.84 0)
 			(effects
@@
 			)
 		)
-		(property "Datasheet" "~"
+		(property "Datasheet" "200mA / 450mΩ"
 			(at 39.37 71.12 0)
 			(effects
@@
 			)
 		)
-		(property "Value" "0u1"
+		(property "Value" "1u"
 			(at 49.53 73.152 0)
 			(effects
@@
 			)
 		)
-		(property "Datasheet" "50V"
+		(property "Datasheet" "25V"
 			(at 49.53 74.93 0)
 			(effects
@@
 			)
 		)
-		(property "LCSC" "C307331"
+		(property "LCSC" "C52923"
 			(at 49.53 74.93 0)
 			(effects
@@
 			)
 		)
-		(property "Value" "0u1"
+		(property "Value" "1u"
 			(at 49.53 118.872 0)
 			(effects
@@
 			)
 		)
-		(property "Datasheet" "50V"
+		(property "Datasheet" "25V"
 			(at 49.53 120.65 0)
 			(effects
@@
 			)
 		)
-		(property "LCSC" "C307331"
+		(property "LCSC" "C52923"
 			(at 49.53 120.65 0)
 			(effects

Commit message: About to delete scan...
Parts:
- U31, U36: Stock (none) -> 15
Other:
- moved on the sheet: L31, L32
Changed lines of the file:
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@@
+	(wire
+		(pts
+			(xy 41.91 71.12) (xy 43.18 71.12)
+		)
+		(stroke
+			(width 0)
+			(type default)
+		)
+	)
 	(wire
 		(pts
@@
 	(wire
 		(pts
-			(xy 33.02 116.84) (xy 35.56 116.84)
+			(xy 31.75 116.84) (xy 34.29 116.84)
 		)
 		(stroke
@@
 	(wire
 		(pts
-			(xy 34.29 71.12) (xy 35.56 71.12)
+			(xy 31.75 71.12) (xy 34.29 71.12)
 		)
 		(stroke
@@
 		(pts
 			(xy 119.38 106.68) (xy 110.49 106.68)
+		)
+		(stroke
+			(width 0)
+			(type default)
+		)
+	)
+	(wire
+		(pts
+			(xy 41.91 116.84) (xy 43.18 116.84)
 		)
 		(stroke
@@
 			)
 		)
+		(property "Stock" ""
+			(at 66.04 66.04 0)
+			(effects
+				(font
+					(size 1.27 1.27)
+				)
+				(hide yes)
+			)
+		)
 		(pin "18"
 		)
@@
 			)
 		)
+		(property "Stock" ""
+			(at 119.38 114.3 0)
+			(effects
+				(font
+					(size 1.27 1.27)
+				)
+				(hide yes)
+			)
+		)
 		(pin "2"
 		)
@@
 	(symbol
 		(lib_id "Parts:+3V3A")
-		(at 33.02 116.84 0)
+		(at 31.75 116.84 0)
 		(unit 1)
 		(exclude_from_sim no)
@@
 		(dnp no)
 		(property "Reference" "#PWR0732"
-			(at 33.02 120.65 0)
+			(at 31.75 120.65 0)
 			(effects
 				(font
@@
 		)
 		(property "Value" "+3V3A"
-			(at 33.02 113.284 0)
+			(at 31.75 113.284 0)
 			(do_not_autoplace yes)
 			(effects
@@
 		)
 		(property "Footprint" ""
-			(at 33.02 116.84 0)
+			(at 31.75 116.84 0)
 			(effects
 				(font
@@
 		)
 		(property "Datasheet" ""
-			(at 33.02 116.84 0)
+			(at 31.75 116.84 0)
 			(effects
 				(font
@@
 		)
 		(property "Description" "Power symbol creates a global label with name {dblquote}+3V3A{dblquote}"
-			(at 33.02 116.84 0)
+			(at 31.75 116.84 0)
 			(effects
 				(font
@@
 			)
 		)
+		(property "Stock" ""
+			(at 66.04 111.76 0)
+			(effects
+				(font
+					(size 1.27 1.27)
+				)
+				(hide yes)
+			)
+		)
 		(pin "18"
 		)
@@
 	(symbol
 		(lib_id "Parts:L_Ferrite_Power")
-		(at 39.37 116.84 90)
+		(at 38.1 116.84 90)
 		(unit 1)
 		(exclude_from_sim no)
@@
 		(dnp no)
 		(property "Reference" "L32"
-			(at 39.37 118.11 90)
+			(at 38.1 118.11 90)
 			(effects
 				(font
@@
 		)
 		(property "Value" "600"
-			(at 39.37 114.046 90)
+			(at 38.1 114.046 90)
 			(effects
 				(font
@@
 		)
 		(property "Footprint" "Inductor_SMD:L_0603_1608Metric"
-			(at 39.37 116.84 0)
+			(at 38.1 116.84 0)
 			(effects
 				(font
@@
 		)
 		(property "Datasheet" "200mA / 450mΩ"
-			(at 39.37 116.84 0)
+			(at 38.1 116.84 0)
 			(effects
 				(font
@@
 		)
 		(property "Description" "Inductor with ferrite core"
-			(at 39.37 116.84 0)
+			(at 38.1 116.84 0)
 			(effects
 				(font
@@
 		)
 		(property "LCSC" "C1002"
-			(at 39.37 116.84 90)
+			(at 38.1 116.84 90)
+			(effects
+				(font
+					(size 1.27 1.27)
+				)
+				(hide yes)
+			)
+		)
+		(property "Stock" ""
+			(at 38.1 116.84 90)
 			(effects
 				(font
@@
 	(symbol
 		(lib_id "Parts:L_Ferrite_Power")
-		(at 39.37 71.12 90)
+		(at 38.1 71.12 90)
 		(unit 1)
 		(exclude_from_sim no)
@@
 		(dnp no)
 		(property "Reference" "L31"
-			(at 39.37 72.39 90)
+			(at 38.1 72.39 90)
 			(effects
 				(font
@@
 		)
 		(property "Value" "600"
-			(at 39.37 68.326 90)
+			(at 38.1 68.326 90)
 			(effects
 				(font
@@
 		)
 		(property "Footprint" "Inductor_SMD:L_0603_1608Metric"
-			(at 39.37 71.12 0)
+			(at 38.1 71.12 0)
 			(effects
 				(font
@@
 		)
 		(property "Datasheet" "200mA / 450mΩ"
-			(at 39.37 71.12 0)
+			(at 38.1 71.12 0)
 			(effects
 				(font
@@
 		)
 		(property "Description" "Inductor with ferrite core"
-			(at 39.37 71.12 0)
+			(at 38.1 71.12 0)
 			(effects
 				(font
@@
 		)
 		(property "LCSC" "C1002"
-			(at 39.37 71.12 90)
+			(at 38.1 71.12 90)
+			(effects
+				(font
+					(size 1.27 1.27)
+				)
+				(hide yes)
+			)
+		)
+		(property "Stock" ""
+			(at 38.1 71.12 90)
 			(effects
 				(font
@@
 			)
 		)
+		(property "Stock" ""
+			(at 43.18 74.93 0)
+			(effects
+				(font
+					(size 1.27 1.27)
+				)
+				(hide yes)
+			)
+		)
 		(pin "1"
 		)
@@
 		)
 		(property "LCSC" "C307331"
+			(at 119.38 68.58 0)
+			(effects
+				(font
+					(size 1.27 1.27)
+				)
+				(hide yes)
+			)
+		)
+		(property "Stock" ""
 			(at 119.38 68.58 0)
 			(effects
@@
 			)
 		)
+		(property "Stock" "15"
+			(at 110.49 114.3 0)
+			(effects
+				(font
+					(size 1.27 1.27)
+				)
+				(hide yes)
+			)
+		)
 		(pin "1"
 		)
@@
 			)
 		)
+		(property "Stock" "15"
+			(at 110.49 68.58 0)
+			(effects
+				(font
+					(size 1.27 1.27)
+				)
+				(hide yes)
+			)
+		)
 		(pin "1"
 		)
@@
 			)
 		)
+		(property "Stock" ""
+			(at 49.53 74.93 0)
+			(effects
+				(font
+					(size 1.27 1.27)
+				)
+				(hide yes)
+			)
+		)
 		(pin "2"
 		)
@@
 			)
 		)
+		(property "Stock" ""
+			(at 43.18 120.65 0)
+			(effects
+				(font
+					(size 1.27 1.27)
+				)
+				(hide yes)
+			)
+		)
 		(pin "1"
 		)
@@
 	(symbol
 		(lib_id "Parts:+3V3A")
-		(at 34.29 71.12 0)
+		(at 31.75 71.12 0)
 		(unit 1)
 		(exclude_from_sim no)
@@
 		(dnp no)
 		(property "Reference" "#PWR0731"
-			(at 34.29 74.93 0)
+			(at 31.75 74.93 0)
 			(effects
 				(font
@@
 		)
 		(property "Value" "+3V3A"
-			(at 34.29 67.564 0)
+			(at 31.75 67.564 0)
 			(do_not_autoplace yes)
 			(effects
@@
 		)
 		(property "Footprint" ""
-			(at 34.29 71.12 0)
+			(at 31.75 71.12 0)
 			(effects
 				(font
@@
 		)
 		(property "Datasheet" ""
-			(at 34.29 71.12 0)
+			(at 31.75 71.12 0)
 			(effects
 				(font
@@
 		)
 		(property "Description" "Power symbol creates a global label with name {dblquote}+3V3A{dblquote}"
-			(at 34.29 71.12 0)
+			(at 31.75 71.12 0)
 			(effects
 				(font
@@
 			(at 49.53 120.65 0)
 			(effects
+				(font
+					(size 1.27 1.27)
+				)
+				(hide yes)
+			)
+		)
+		(property "Stock" ""
+			(at 49.53 120.65 0)
+			(effects

Commit message: Most blocks there....
About to restore scan.
Parts:
- added C387, C388, C389, C390: 1u, Capacitor_SMD:C_0402_1005Metric, symbol Device:C
- added U34, U39: OPA2388DGK, Parts:OPA2388, symbol Parts:OPA2388DGK
Connections:
- net GNDPWR: now also C387.2, C388.1, C389.2, C390.1
- new net +2V5: C387.1, C389.1, U34.8 (V+), U39.8 (V+)
- new net -2V5: C388.2, C390.2, U34.4 (V-), U39.4 (V-)
Other:
- moved on the sheet: C382, C384, U31C, U36C
