File: common2752.kicad_sch (KiCad schematic)
At the start: 18 parts, among them U30 LTC2752B, U31 OPA2189DGK, U34 OPA2388DGK, U35 LTC2752B, U36 OPA2189DGK, U39 OPA2388DGK

Commit message: Tweak various feedback loops.
Parts:
- H31, H32, H33, H34: Stock (none) -> Board
- U34, U39: Stock 14 -> 14+LCSC
Changed lines of the file:
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@@
+			)
+		)
+		(property "Stock" "Board"
+			(at 104.14 88.9 0)
+			(effects
+				(font
+					(size 1.27 1.27)
+				)
+				(hide yes)
 			)
 		)
@@
 			)
 		)
-		(property "Sim.Library" "spice/opa2388.lib"
-			(at 130.81 111.76 0)
-			(effects
-				(font
-					(size 1.27 1.27)
-				)
-				(hide yes)
-			)
-		)
-		(property "Sim.Name" "OPA2388"
-			(at 130.81 111.76 0)
-			(effects
-				(font
-					(size 1.27 1.27)
-				)
-				(hide yes)
-			)
-		)
-		(property "Sim.Device" "SUBCKT"
-			(at 130.81 111.76 0)
-			(effects
-				(font
-					(size 1.27 1.27)
-				)
-				(hide yes)
-			)
-		)
-		(property "Sim.Pins" "1=aout 2=a- 3=a+ 4=v- 5=b+ 6=b- 7=bout 8=v+"
-			(at 130.81 111.76 0)
-			(effects
-				(font
-					(size 1.27 1.27)
-				)
-				(hide yes)
-			)
-		)
-		(property "Stock" "14"
+		(property "Stock" "14+LCSC"
 			(at 130.81 111.76 0)
 			(effects
@@
 			)
 		)
+		(property "Stock" "Board"
+			(at 99.06 88.9 0)
+			(effects
+				(font
+					(size 1.27 1.27)
+				)
+				(hide yes)
+			)
+		)
 		(instances
 			(project "lincal"
@@
 		)
 		(property "Description" "Mounting Hole without connection"
+			(at 93.98 88.9 0)
+			(effects
+				(font
+					(size 1.27 1.27)
+				)
+				(hide yes)
+			)
+		)
+		(property "Stock" "Board"
 			(at 93.98 88.9 0)
 			(effects
@@
 			)
 		)
-		(property "Sim.Library" "spice/opa2388.lib"
-			(at 132.08 66.04 0)
-			(effects
-				(font
-					(size 1.27 1.27)
-				)
-				(hide yes)
-			)
-		)
-		(property "Sim.Name" "OPA2388"
-			(at 132.08 66.04 0)
-			(effects
-				(font
-					(size 1.27 1.27)
-				)
-				(hide yes)
-			)
-		)
-		(property "Sim.Device" "SUBCKT"
-			(at 132.08 66.04 0)
-			(effects
-				(font
-					(size 1.27 1.27)
-				)
-				(hide yes)
-			)
-		)
-		(property "Sim.Pins" "1=aout 2=a- 3=a+ 4=v- 5=b+ 6=b- 7=bout 8=v+"
-			(at 132.08 66.04 0)
-			(effects
-				(font
-					(size 1.27 1.27)
-				)
-				(hide yes)
-			)
-		)
-		(property "Stock" "14"
+		(property "Stock" "14+LCSC"
 			(at 132.08 66.04 0)
 			(effects
@@
 			(at 88.9 88.9 0)
 			(effects
+				(font
+					(size 1.27 1.27)
+				)
+				(hide yes)
+			)
+		)
+		(property "Stock" "Board"
+			(at 88.9 88.9 0)
+			(effects
