File: lincal.kicad_sch (KiCad schematic)
At the start: 0 parts

Commit message: Redo the reference ground star point.
Other:
- sheet Reference ports: added AGNDsh1, AGNDsh2; removed none
- sheet Sample Hold 1 ports: added AGND; removed none
- sheet Sample Hold 2 ports: added AGND; removed none
Changed lines of the file:
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@@
+	(wire
+		(pts
+			(xy 97.79 102.87) (xy 106.68 102.87)
+		)
+		(stroke
+			(width 0)
+			(type default)
+		)
+	)
+	(wire
+		(pts
+			(xy 106.68 105.41) (xy 97.79 105.41)
+		)
+		(stroke
+			(width 0)
+			(type default)
+		)
+	)
 	(wire
 		(pts
@@
 	(wire
 		(pts
+			(xy 106.68 119.38) (xy 116.84 119.38)
+		)
+		(stroke
+			(width 0)
+			(type default)
+		)
+	)
+	(wire
+		(pts
 			(xy 106.68 62.23) (xy 97.79 62.23)
 		)
@@
 	(wire
 		(pts
+			(xy 106.68 83.82) (xy 97.79 83.82)
+		)
+		(stroke
+			(width 0)
+			(type default)
+		)
+	)
+	(wire
+		(pts
 			(xy 62.23 146.05) (xy 53.34 146.05)
 		)
@@
 	(wire
 		(pts
+			(xy 106.68 121.92) (xy 116.84 121.92)
+		)
+		(stroke
+			(width 0)
+			(type default)
+		)
+	)
+	(wire
+		(pts
 			(xy 166.37 71.12) (xy 157.48 71.12)
 		)
@@
 	(wire
 		(pts
-			(xy 97.79 83.82) (xy 106.68 83.82)
+			(xy 97.79 81.28) (xy 106.68 81.28)
 		)
 		(stroke
@@
 		(pts
 			(xy 62.23 151.13) (xy 53.34 151.13)
-		)
-		(stroke
-			(width 0)
-			(type default)
-		)
-	)
-	(wire
-		(pts
-			(xy 97.79 105.41) (xy 106.68 105.41)
 		)
 		(stroke
@@
 		)
 	)
+	(label "AGNDsh2"
+		(at 116.84 121.92 180)
+		(effects
+			(font
+				(size 1.27 1.27)
+			)
+			(justify right bottom)
+		)
+	)
 	(label "Sample2"
-		(at 97.79 105.41 0)
+		(at 97.79 102.87 0)
 		(effects
 			(font
@@
 	)
 	(label "Sample1"
-		(at 97.79 83.82 0)
+		(at 97.79 81.28 0)
 		(effects
 			(font
@@
 		)
 	)
+	(label "AGNDsh1"
+		(at 116.84 119.38 180)
+		(effects
+			(font
+				(size 1.27 1.27)
+			)
+			(justify right bottom)
+		)
+	)
 	(label "OffsetA1"
 		(at 157.48 90.17 0)
@@
 		)
 	)
+	(label "AGNDsh1"
+		(at 97.79 83.82 0)
+		(effects
+			(font
+				(size 1.27 1.27)
+			)
+			(justify left bottom)
+		)
+	)
 	(label "SCK"
 		(at 157.48 62.23 0)
@@
 			)
 			(justify right bottom)
+		)
+	)
+	(label "AGNDsh2"
+		(at 97.79 105.41 0)
+		(effects
+			(font
+				(size 1.27 1.27)
+			)
+			(justify left bottom)
 		)
 	)
@@
 	)
 	(sheet
-		(at 91.44 116.84)
-		(size 15.24 5.08)
+		(at 91.44 115.57)
+		(size 15.24 7.62)
 		(exclude_from_sim no)
 		(in_bom yes)
@@
 		)
 		(property "Sheetname" "Reference"
-			(at 91.694 118.872 0)
+			(at 91.694 117.602 0)
 			(effects
 				(font
@@
 		)
 		(property "Sheetfile" "ref.kicad_sch"
-			(at 91.44 122.5046 0)
+			(at 91.44 123.7746 0)
 			(effects
 				(font
@@
 				)
 				(justify left top)
+			)
+		)
+		(pin "AGNDsh1" passive
+			(at 106.68 119.38 0)
+			(effects
+				(font
+					(size 1.27 1.27)
+				)
+				(justify right)
+			)
+		)
+		(pin "AGNDsh2" passive
+			(at 106.68 121.92 0)
+			(effects
+				(font
+					(size 1.27 1.27)
+				)
+				(justify right)
 			)
 		)
@@
 		)
 		(pin "Sample" input
-			(at 106.68 105.41 180)
+			(at 106.68 102.87 180)
 			(effects
 				(font
@@
 				)
 				(justify right)
+			)
+		)
+		(pin "AGND" passive
+			(at 106.68 105.41 180)
+			(effects
+				(font
+					(size 1.27 1.27)
+				)
+				(justify left)
 			)
 		)
@@
 	)
 	(sheet
-		(at 113.03 116.84)
+		(at 128.27 116.84)
 		(size 13.97 5.08)
 		(exclude_from_sim no)
@@
 		)
 		(property "Sheetname" "18V"
-			(at 113.538 118.872 0)
+			(at 128.778 118.872 0)
 			(effects
 				(font
@@
 		)
 		(property "Sheetfile" "v18.kicad_sch"
-			(at 113.03 122.7586 0)
+			(at 128.27 122.7586 0)
 			(effects
 				(font
@@
 		)
 		(pin "Sample" input
-			(at 106.68 83.82 180)
+			(at 106.68 81.28 180)
 			(effects
 				(font
@@
 				)
 				(justify right)
+			)
+		)
+		(pin "AGND" passive
+			(at 106.68 83.82 180)
+			(effects
+				(font
+					(size 1.27 1.27)
+				)
+				(justify left)
 			)
 		)
@@
 	)
 	(sheet
-		(at 133.35 116.84)
+		(at 148.59 116.84)
 		(size 13.97 5.08)
 		(exclude_from_sim no)
@@
 		)
 		(property "Sheetname" "Low Voltage"
-			(at 133.858 119.126 0)
+			(at 149.098 119.126 0)
 			(effects
 				(font
@@
 		)
 		(property "Sheetfile" "power.kicad_sch"
-			(at 133.35 122.5046 0)
-			(effects
-				(font
+			(at 148.59 122.5046 0)
+			(effects
+				(font

Commit message: Remove placebo planes.  Tidy some analog routing.
Other:
- sheet Reference ports: added none; removed AGNDsh1, AGNDsh2
- sheet Sample Hold 1 ports: added none; removed AGND
- sheet Sample Hold 2 ports: added none; removed AGND
Changed lines of the file:
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@@
-	(wire
-		(pts
-			(xy 106.68 105.41) (xy 97.79 105.41)
-		)
-		(stroke
-			(width 0)
-			(type default)
-		)
-	)
 	(wire
 		(pts
@@
 	(wire
 		(pts
-			(xy 106.68 119.38) (xy 116.84 119.38)
-		)
-		(stroke
-			(width 0)
-			(type default)
-		)
-	)
-	(wire
-		(pts
 			(xy 106.68 62.23) (xy 97.79 62.23)
 		)
@@
 	(wire
 		(pts
-			(xy 106.68 83.82) (xy 97.79 83.82)
-		)
-		(stroke
-			(width 0)
-			(type default)
-		)
-	)
-	(wire
-		(pts
 			(xy 62.23 146.05) (xy 53.34 146.05)
 		)
@@
 		(pts
 			(xy 57.15 73.66) (xy 58.42 73.66)
-		)
-		(stroke
-			(width 0)
-			(type default)
-		)
-	)
-	(wire
-		(pts
-			(xy 106.68 121.92) (xy 116.84 121.92)
 		)
 		(stroke
@@
 		)
 	)
-	(label "AGNDsh2"
-		(at 116.84 121.92 180)
-		(effects
-			(font
-				(size 1.27 1.27)
-			)
-			(justify right bottom)
-		)
-	)
 	(label "Sample2"
 		(at 97.79 102.87 0)
@@
 		)
 	)
-	(label "AGNDsh1"
-		(at 116.84 119.38 180)
-		(effects
-			(font
-				(size 1.27 1.27)
-			)
-			(justify right bottom)
-		)
-	)
 	(label "OffsetA1"
 		(at 157.48 90.17 0)
@@
 		)
 	)
-	(label "AGNDsh1"
-		(at 97.79 83.82 0)
-		(effects
-			(font
-				(size 1.27 1.27)
-			)
-			(justify left bottom)
-		)
-	)
 	(label "SCK"
 		(at 157.48 62.23 0)
@@
 			)
 			(justify right bottom)
-		)
-	)
-	(label "AGNDsh2"
-		(at 97.79 105.41 0)
-		(effects
-			(font
-				(size 1.27 1.27)
-			)
-			(justify left bottom)
 		)
 	)
@@
 	)
 	(sheet
-		(at 91.44 115.57)
-		(size 15.24 7.62)
+		(at 92.71 116.84)
+		(size 15.24 5.08)
 		(exclude_from_sim no)
 		(in_bom yes)
@@
 		)
 		(property "Sheetname" "Reference"
-			(at 91.694 117.602 0)
+			(at 92.964 118.872 0)
 			(effects
 				(font
@@
 		)
 		(property "Sheetfile" "ref.kicad_sch"
-			(at 91.44 123.7746 0)
+			(at 92.71 122.7586 0)
 			(effects
 				(font
@@
 				)
 				(justify left top)
-			)
-		)
-		(pin "AGNDsh1" passive
-			(at 106.68 119.38 0)
-			(effects
-				(font
-					(size 1.27 1.27)
-				)
-				(justify right)
-			)
-		)
-		(pin "AGNDsh2" passive
-			(at 106.68 121.92 0)
-			(effects
-				(font
-					(size 1.27 1.27)
-				)
-				(justify right)
 			)
 		)
@@
 			)
 		)
-		(pin "AGND" passive
-			(at 106.68 105.41 180)
-			(effects
-				(font
-					(size 1.27 1.27)
-				)
-				(justify left)
-			)
-		)
 		(instances
 			(project "lincal"
@@
 	)
 	(sheet
-		(at 128.27 116.84)
+		(at 114.3 116.84)
 		(size 13.97 5.08)
 		(exclude_from_sim no)
@@
 		)
 		(property "Sheetname" "18V"
-			(at 128.778 118.872 0)
+			(at 114.808 118.872 0)
 			(effects
 				(font
@@
 		)
 		(property "Sheetfile" "v18.kicad_sch"
-			(at 128.27 122.7586 0)
+			(at 114.3 122.7586 0)
 			(effects
 				(font
@@
 			)
 		)
-		(pin "AGND" passive
-			(at 106.68 83.82 180)
-			(effects
-				(font
-					(size 1.27 1.27)
-				)
-				(justify left)
-			)
-		)
 		(instances
 			(project "lincal"
@@
 	)
 	(sheet
-		(at 148.59 116.84)
+		(at 134.62 116.84)
 		(size 13.97 5.08)
 		(exclude_from_sim no)
@@
 		)
 		(property "Sheetname" "Low Voltage"
-			(at 149.098 119.126 0)
+			(at 135.128 119.126 0)
 			(effects
 				(font
@@
 		)
 		(property "Sheetfile" "power.kicad_sch"
-			(at 148.59 122.5046 0)
-			(effects
-				(font
+			(at 134.62 122.5046 0)
+			(effects
+				(font
