File: lincal.kicad_sch (KiCad schematic)
At the start: 0 parts

Commit message: Readyish
Parts:
- added J10: Scan2, Parts:TestPoint, symbol Connector:Conn_01x01_Socket
- added J21, J22: DAC1A, Parts:TestPoint, symbol Connector:Conn_01x01_Socket
- added J23: DAC2A, Parts:TestPoint, symbol Connector:Conn_01x01_Socket
- added J24: DAC2B, Parts:TestPoint, symbol Connector:Conn_01x01_Socket
- added J8: Offset, Parts:TestPoint, symbol Connector:Conn_01x01_Socket
- added J9: Scan1, Parts:TestPoint, symbol Connector:Conn_01x01_Socket
Connections:
- net DAC1A: now also J21.1 (Pin_1)
- net DAC1B: now also J22.1 (Pin_1)
- net DAC2A: now also J23.1 (Pin_1)
- net DAC2B: now also J24.1 (Pin_1)
- net Offset: now also J8.1 (Pin_1)
- net Scan1: now also J9.1 (Pin_1)
- net Scan2: now also J10.1 (Pin_1)
