File: ref.kicad_sch (KiCad schematic)
At the start: 43 parts, among them Q61 BSS139, U6 REF7050, U61 OPA2189DGK, U62 OPA828DGN

Commit message: More component metadata.
Parts:
- C61, C62, C63, C64, C65, C66, C67, C68, C69, C70, C71, C73, L61, R608, R611, R66, R67, R70, R72, U6, U62: Stock (none) -> JLC
- NT61: Stock (none) -> Board
- Q61: Stock (none) -> ?; now left out of the parts list
- R60: LCSC (none) -> C25811; Stock (none) -> JLC
- R601, R602, R603, R604, R605, R606, R61, R62, R63: Stock (none) -> Digikey
- R64: Stock (none) -> JLC; now in the parts list
- R68: LCSC (none) -> C22843; Stock (none) -> JLC
- R69: Stock (none) -> 50
- TP61, TP62, TP63, TP64, TP66: Stock - -> Board
Changed lines of the file:
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@@
 			)
 		)
-		(property "LCSC" ""
+		(property "LCSC" "C25811"
 			(at 148.59 54.61 90)
 			(effects
@@
 			)
 		)
-		(property "Stock" ""
+		(property "Stock" "JLC"
 			(at 148.59 54.61 90)
 			(effects
@@
 			)
 		)
-		(property "Stock" ""
+		(property "Stock" "Digikey"
 			(at 176.53 71.12 90)
 			(effects
@@
 			)
 		)
-		(property "Stock" ""
+		(property "Stock" "JLC"
 			(at 138.43 120.65 0)
 			(effects
@@
 			)
 		)
-		(property "Stock" ""
+		(property "Stock" "Digikey"
 			(at 180.34 101.6 90)
 			(effects
@@
 			)
 		)
-		(property "Stock" ""
+		(property "Stock" "JLC"
 			(at 143.51 85.09 90)
 			(effects
@@
 			)
 		)
-		(property "Stock" ""
+		(property "Stock" "JLC"
 			(at 83.82 55.88 0)
 			(effects
@@
 			)
 		)
-		(property "Stock" "-"
+		(property "Stock" "Board"
 			(at 191.77 57.15 0)
 			(effects
@@
 			)
 		)
-		(property "Stock" ""
+		(property "Stock" "JLC"
 			(at 144.78 124.46 90)
 			(effects
@@
 			)
 		)
-		(property "Stock" ""
+		(property "Stock" "JLC"
 			(at 168.91 54.61 90)
 			(effects
@@
 			)
 		)
-		(property "Stock" ""
+		(property "Stock" "JLC"
 			(at 63.5 52.07 90)
 			(effects
@@
 			)
 		)
-		(property "Stock" ""
+		(property "Stock" "JLC"
 			(at 152.4 120.65 0)
 			(effects
@@
 			)
 		)
-		(property "Stock" ""
+		(property "Stock" "JLC"
 			(at 133.35 85.09 90)
 			(effects
@@
 			)
 		)
-		(property "Stock" ""
+		(property "Stock" "JLC"
 			(at 187.96 71.12 90)
 			(effects
@@
 			)
 		)
-		(property "Stock" "-"
+		(property "Stock" "Board"
 			(at 83.82 52.07 0)
 			(effects
@@
 			)
 		)
-		(property "Stock" ""
+		(property "Stock" "Digikey"
 			(at 180.34 81.28 90)
 			(effects
@@
 			)
 		)
-		(property "Stock" ""
+		(property "Stock" "Digikey"
 			(at 176.53 68.58 90)
 			(effects
@@
 			)
 		)
-		(property "Stock" ""
+		(property "Stock" "JLC"
 			(at 97.79 57.15 0)
 			(effects
@@
 			)
 		)
-		(property "Stock" "-"
+		(property "Stock" "Board"
 			(at 111.76 52.07 0)
 			(effects
@@
 			)
 		)
-		(property "Stock" ""
+		(property "Stock" "JLC"
 			(at 175.26 76.2 0)
 			(effects
@@
 			)
 		)
-		(property "Stock" ""
+		(property "Stock" "Board"
 			(at 100.33 67.31 0)
 			(effects
@@
 			)
 		)
-		(property "Stock" ""
+		(property "Stock" "JLC"
 			(at 175.26 96.52 0)
 			(effects
@@
 			)
 		)
-		(property "Stock" ""
+		(property "Stock" "Digikey"
 			(at 180.34 111.76 90)
 			(effects
@@
 			)
 		)
-		(property "Stock" ""
+		(property "Stock" "JLC"
 			(at 83.82 106.68 0)
 			(effects
@@
 			)
 		)
+		(property "Stock" "JLC"
+			(at 180.34 57.15 0)
+			(effects
+				(font
+					(size 1.27 1.27)
+				)
+				(hide yes)
+			)
+		)
 		(pin "3"
 		)
@@
 			)
 		)
-		(property "Stock" ""
+		(property "Stock" "JLC"
 			(at 116.84 55.88 0)
 			(effects
@@
 			)
 		)
-		(property "Stock" ""
+		(property "Stock" "JLC"
 			(at 175.26 106.68 0)
 			(effects
@@
 			)
 		)
-		(property "Stock" "-"
+		(property "Stock" "Board"
 			(at 143.51 54.61 0)
 			(effects
@@
 		(unit 1)
 		(exclude_from_sim no)
-		(in_bom yes)
+		(in_bom no)
 		(on_board yes)
 		(dnp no)
@@
 			)
 		)
+		(property "Stock" "?"
+			(at 161.29 52.07 90)
+			(effects
+				(font
+					(size 1.27 1.27)
+				)
+				(hide yes)
+			)
+		)
 		(pin "2"
 		)
@@
 			)
 		)
-		(property "Stock" ""
+		(property "Stock" "50"
 			(at 185.42 118.11 90)
 			(effects
@@
 			)
 		)
-		(property "Stock" ""
+		(property "Stock" "JLC"
 			(at 77.47 55.88 0)
 			(effects
@@
 			)
 		)
-		(property "Stock" ""
+		(property "Stock" "JLC"
 			(at 144.78 116.84 90)
 			(effects
@@
 			)
 		)
-		(property "Stock" ""
+		(property "Stock" "Digikey"
 			(at 180.34 91.44 90)
 			(effects
@@
 		(unit 1)
 		(exclude_from_sim no)
-		(in_bom no)
+		(in_bom yes)
 		(on_board yes)
 		(dnp no)
@@
 			)
 		)
-		(property "Stock" ""
+		(property "Stock" "JLC"
 			(at 71.12 52.07 90)
 			(effects
@@
 			)
 		)
-		(property "Stock" ""
+		(property "Stock" "JLC"
 			(at 76.2 106.68 0)
 			(effects
@@
 			)
 		)
-		(property "Datasheet" "~"
+		(property "Datasheet" "Swappable"
 			(at 175.26 118.11 0)
 			(effects
@@
 			)
 		)
-		(property "LCSC" ""
+		(property "LCSC" "C22843"
 			(at 175.26 118.11 90)
 			(effects
@@
 			)
 		)
-		(property "Stock" ""
+		(property "Stock" "JLC"
 			(at 175.26 118.11 90)
 			(effects
@@
 			)
 		)
-		(property "Stock" ""
+		(property "Stock" "Digikey"
 			(at 138.43 59.69 90)
 			(effects
@@
 			)
 		)
-		(property "Stock" ""
+		(property "Stock" "JLC"
 			(at 111.76 55.88 0)
 			(effects
@@
 			)
 		)
-		(property "Stock" ""
+		(property "Stock" "Digikey"
 			(at 138.43 80.01 90)
 			(effects
@@
 			)
 		)
-		(property "Stock" ""
+		(property "Stock" "Digikey"
 			(at 138.43 69.85 90)
 			(effects
@@
 			)
 		)
-		(property "Stock" ""
+		(property "Stock" "JLC"
 			(at 175.26 86.36 0)
 			(effects
@@
 			)
 		)
-		(property "Stock" "-"
+		(property "Stock" "Board"
 			(at 116.84 74.93 0)
 			(effects

Commit message: Front panel
Parts:
- AGND1: renamed from TP63; value GND -> AGND
- R608: value 100 -> 150
- renumbered TP64 to Raw15, TP62 to Raw5, TP66 to Ref15, TP61 to RefIn1
Connections:
- net GND: no longer C61.2
- net at C62.2, NT61.1, U6.3 (GND)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: now also C61.2
- net rin renamed Rin
Changed lines of the file:
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@@
 	)
 	(junction
+		(at 83.82 67.31)
+		(diameter 0)
+		(color 0 0 0 0)
+	)
+	(junction
 		(at 83.82 99.06)
 		(diameter 0)
@@
 	(wire
 		(pts
+			(xy 77.47 59.69) (xy 77.47 67.31)
+		)
+		(stroke
+			(width 0)
+			(type default)
+		)
+	)
+	(wire
+		(pts
 			(xy 138.43 54.61) (xy 138.43 55.88)
 		)
@@
 	(wire
 		(pts
+			(xy 77.47 67.31) (xy 83.82 67.31)
+		)
+		(stroke
+			(width 0)
+			(type default)
+		)
+	)
+	(wire
+		(pts
 			(xy 147.32 85.09) (xy 148.59 85.09)
 		)
@@
 		(effects
 			(font
-				(face "Liberation Mono")
-				(size 1.27 1.27)
+				(size 1.016 1.016)
 			)
 			(justify left bottom)
 		)
 	)
-	(label "rin"
+	(label "Rin"
 		(at 80.01 52.07 0)
 		(effects
 			(font
-				(size 1.27 1.27)
+				(size 1.016 1.016)
 			)
 			(justify left bottom)
@@
 		(effects
 			(font
-				(face "Liberation Mono")
-				(size 1.27 1.27)
+				(size 1.016 1.016)
 			)
 			(justify right bottom)
@@
 		(effects
 			(font
-				(size 1.27 1.27)
+				(size 1.016 1.016)
 			)
 			(justify bottom)
@@
 		(on_board yes)
 		(dnp no)
-		(property "Reference" "TP66"
-			(at 191.77 51.816 0)
+		(property "Reference" "Ref15"
+			(at 192.786 52.07 0)
 			(effects
 				(font
@@
 			(project "lincal"
 				(path "/b054cef4-39e3-49d8-aff0-7ba5a206c187/525413b8-c4e9-4b1d-b0c6-ca0be2e26a7f"
-					(reference "TP66")
+					(reference "Ref15")
 					(unit 1)
 				)
@@
 			)
 		)
-		(property "Value" "100"
+		(property "Value" "150"
 			(at 168.91 54.61 90)
 			(effects
@@
 		(on_board yes)
 		(dnp no)
-		(property "Reference" "TP61"
+		(property "Reference" "RefIn1"
 			(at 83.82 46.736 0)
 			(effects
@@
 			(project "lincal"
 				(path "/b054cef4-39e3-49d8-aff0-7ba5a206c187/525413b8-c4e9-4b1d-b0c6-ca0be2e26a7f"
-					(reference "TP61")
+					(reference "RefIn1")
 					(unit 1)
 				)
@@
 		(on_board yes)
 		(dnp no)
-		(property "Reference" "TP62"
+		(property "Reference" "Raw5"
 			(at 111.76 46.736 0)
 			(effects
@@
 					(size 1.27 1.27)
 				)
+				(hide yes)
 			)
 		)
@@
 					(size 1.27 1.27)
 				)
-				(hide yes)
 			)
 		)
@@
 			(project "lincal"
 				(path "/b054cef4-39e3-49d8-aff0-7ba5a206c187/525413b8-c4e9-4b1d-b0c6-ca0be2e26a7f"
-					(reference "TP62")
+					(reference "Raw5")
 					(unit 1)
 				)
@@
 	)
 	(symbol
-		(lib_id "power:GND")
-		(at 77.47 59.69 0)
-		(unit 1)
-		(exclude_from_sim no)
-		(in_bom yes)
-		(on_board yes)
-		(dnp no)
-		(property "Reference" "#PWR0253"
-			(at 77.47 66.04 0)
-			(effects
-				(font
-					(size 1.27 1.27)
-				)
-				(hide yes)
-			)
-		)
-		(property "Value" "GND"
-			(at 77.47 63.5 0)
-			(effects
-				(font
-					(size 1.27 1.27)
-				)
-				(hide yes)
-			)
-		)
-		(property "Footprint" ""
-			(at 77.47 59.69 0)
-			(effects
-				(font
-					(size 1.27 1.27)
-				)
-				(hide yes)
-			)
-		)
-		(property "Datasheet" ""
-			(at 77.47 59.69 0)
-			(effects
-				(font
-					(size 1.27 1.27)
-				)
-				(hide yes)
-			)
-		)
-		(property "Description" "Power symbol creates a global label with name \"GND\" , ground"
-			(at 77.47 59.69 0)
-			(effects
-				(font
-					(size 1.27 1.27)
-				)
-				(hide yes)
-			)
-		)
-		(pin "1"
-		)
-		(instances
-			(project "lincal"
-				(path "/b054cef4-39e3-49d8-aff0-7ba5a206c187/525413b8-c4e9-4b1d-b0c6-ca0be2e26a7f"
-					(reference "#PWR0253")
-					(unit 1)
-				)
-			)
-		)
-	)
-	(symbol
 		(lib_id "Device:NetTie_3_Tee")
 		(at 100.33 67.31 0)
@@
 		(on_board yes)
 		(dnp no)
-		(property "Reference" "TP64"
+		(property "Reference" "Raw15"
 			(at 143.51 49.276 0)
 			(effects
@@
 			(project "lincal"
 				(path "/b054cef4-39e3-49d8-aff0-7ba5a206c187/525413b8-c4e9-4b1d-b0c6-ca0be2e26a7f"
-					(reference "TP64")
+					(reference "Raw15")
 					(unit 1)
 				)
@@
 	)
 	(symbol
+		(lib_id "power:PWR_FLAG")
+		(at 83.82 67.31 180)
+		(unit 1)
+		(exclude_from_sim no)
+		(in_bom yes)
+		(on_board yes)
+		(dnp no)
+		(property "Reference" "#FLG0811"
+			(at 83.82 69.215 0)
+			(effects
+				(font
+					(size 1.27 1.27)
+				)
+				(hide yes)
+			)
+		)
+		(property "Value" "PWR_FLAG"
+			(at 83.82 71.12 0)
+			(effects
+				(font
+					(size 1.27 1.27)
+				)
+				(hide yes)
+			)
+		)
+		(property "Footprint" ""
+			(at 83.82 67.31 0)
+			(effects
+				(font
+					(size 1.27 1.27)
+				)
+				(hide yes)
+			)
+		)
+		(property "Datasheet" "~"
+			(at 83.82 67.31 0)
+			(effects
+				(font
+					(size 1.27 1.27)
+				)
+				(hide yes)
+			)
+		)
+		(property "Description" "Special symbol for telling ERC where power comes from"
+			(at 83.82 67.31 0)
+			(effects
+				(font
+					(size 1.27 1.27)
+				)
+				(hide yes)
+			)
+		)
+		(pin "1"
+		)
+		(instances
+			(project "lincal"
+				(path "/b054cef4-39e3-49d8-aff0-7ba5a206c187/525413b8-c4e9-4b1d-b0c6-ca0be2e26a7f"
+					(reference "#FLG0811")
+					(unit 1)
+				)
+			)
+		)
+	)
+	(symbol
 		(lib_id "power:GNDPWR")
 		(at 100.33 69.85 0)
@@
 		(on_board yes)
 		(dnp no)
-		(property "Reference" "TP63"
+		(property "Reference" "AGND1"
 			(at 116.84 69.596 0)
 			(effects
@@
 			)
 		)
-		(property "Value" "GND"
+		(property "Value" "AGND"
 			(at 116.84 69.85 0)
 			(effects
@@
 			(project "lincal"
 				(path "/b054cef4-39e3-49d8-aff0-7ba5a206c187/525413b8-c4e9-4b1d-b0c6-ca0be2e26a7f"
-					(reference "TP63")
+					(reference "AGND1")
 					(unit 1)
 				)
