File: v18.kicad_sch (KiCad schematic)
At the start: 61 parts, among them U51 ADP5071ACPZ, U52 TPS7A4700xRGW, U53 TPS7A3301RGW

Commit message: Progress checkin.  About to redo FDA feedback again.
Parts:
- added L57, L58: 100, Inductor_SMD:L_0603_1608Metric, symbol Parts:L_Ferrite_Power
- renumbered D57 to D53, D58 to D54, D55 to D56, D56 to D57
Connections:
- net +19V: now also C525.1, C526.1, C527.1, C528.1, C529.1, C530.1; no longer C525.2, C526.2, C527.2, C528.2, C529.2, C530.2
- net +21V: now also L57.2; no longer C505.1, C52.1, D51.1 (K), D53.2 (A), R503.1, TP51.1
- net -18V: now also L58.2; no longer C508.2, C53.2, D52.2 (A), D54.1 (K), R514.2, TP53.1
- net GNDPWR: now also C50.2, C525.2, C526.2, C527.2, C528.2, C529.2, C530.2; no longer C50.1, C525.1, C526.1, C527.1, C528.1, C529.1, C530.1
- net P5V: now also C50.1; no longer C50.2
- new net: C508.2, C53.2, D52.2 (A), D54.1 (K), L58.1, R514.2, TP53.1
- new net: C505.1, C52.1, D51.1 (K), D53.2 (A), L57.1, R503.1, TP51.1
Other:
- moved on the sheet: C50, C525, C526, C527, C528, C529, C530

Commit message: Start to place within physical board size.
Connections:
- net GNDPWR: now also C524.2; no longer C524.1
- net at U52.14 (NR): now also C524.1; no longer C524.2
Changed lines of the file:
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@@
 		(lib_id "Device:C")
 		(at 200.66 72.39 0)
-		(mirror x)
 		(unit 1)
 		(exclude_from_sim no)
@@
 		(dnp no)
 		(property "Reference" "C524"
+			(at 200.66 70.358 0)
+			(effects
+				(font
+					(size 1.27 1.27)
+				)
+				(justify left)
+			)
+		)
+		(property "Value" "1u"
 			(at 200.66 74.422 0)
 			(effects
@@
 			)
 		)
-		(property "Value" "1u"
-			(at 200.66 70.358 0)
-			(effects
-				(font
-					(size 1.27 1.27)
-				)
-				(justify left)
-			)
-		)
 		(property "Footprint" "Capacitor_SMD:C_0402_1005Metric"
-			(at 201.6252 68.58 0)
+			(at 201.6252 76.2 0)
 			(effects
 				(font
@@
 					(size 1.27 1.27)
 				)
-				(justify left)
+				(justify right)
 			)
 		)
@@
 					(size 1.27 1.27)
 				)
-				(justify left)
-			)
-		)
+				(justify right)
+			)
+		)

Commit message: Nearly all routed.  Repinning FDA resistors.
Parts:
- R502: LCSC C23172 -> (none)
- R543: LCSC C25811 -> (none)
Changed lines of the file:
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@@
 			)
 		)
-		(property "LCSC" "C23172"
+		(property "LCSC" ""
 			(at 118.11 59.69 90)
 			(effects
@@
 			)
 		)
-		(property "LCSC" "C25811"
+		(property "LCSC" ""
 			(at 207.01 114.3 90)
 			(effects

Commit message: DRC update.  Repin ADC.  De-crack the S/H ground.
Parts:
- TP51: value TestPoint -> 21V
- TP52: value TestPoint -> 19V
- TP53: value TestPoint -> -18V
- TP54: value TestPoint -> -16V
- U51: footprint Package_CSP:LFCSP-20-1EP_4x4mm_P0.5mm_EP2.6x2.6mm -> Parts:LFCSP-20-1EP_4x4mm_P0.5mm_EP2.6x2.6mm
- U52, U53: footprint Package_DFN_QFN:Texas_RGW0020A_VQFN-20-1EP_5x5mm_P0.65mm_EP3.15x3.15mm -> Parts:Texas_RGW0020A_VQFN-20-1EP_5x5mm_P0.65mm_EP3.15x3.15mm
- renumbered C523 to C54
Changed lines of the file:
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@@
 	)
 	(junction
+		(at 128.27 86.36)
+		(diameter 0)
+		(color 0 0 0 0)
+	)
+	(junction
 		(at 80.01 60.96)
 		(diameter 0)
@@
 	(wire
 		(pts
-			(xy 123.19 86.36) (xy 134.62 86.36)
+			(xy 123.19 86.36) (xy 128.27 86.36)
 		)
 		(stroke
@@
 	(wire
 		(pts
+			(xy 128.27 86.36) (xy 134.62 86.36)
+		)
+		(stroke
+			(width 0)
+			(type default)
+		)
+	)
+	(wire
+		(pts
 			(xy 176.53 76.2) (xy 185.42 76.2)
 		)
@@
 			)
 		)
-		(property "Value" "TestPoint"
+		(property "Value" "-18V"
 			(at 134.62 97.79 0)
 			(effects
@@
 			)
 		)
-		(property "Footprint" "Package_CSP:LFCSP-20-1EP_4x4mm_P0.5mm_EP2.6x2.6mm"
+		(property "Footprint" "Parts:LFCSP-20-1EP_4x4mm_P0.5mm_EP2.6x2.6mm"
 			(at 97.79 88.9 0)
 			(effects
@@
 			)
 		)
-		(property "Value" "TestPoint"
+		(property "Value" "-16V"
 			(at 223.52 87.63 0)
 			(effects
@@
 			)
 		)
-		(property "Value" "TestPoint"
+		(property "Value" "19V"
 			(at 223.52 38.1 0)
 			(effects
@@
 	)
 	(symbol
+		(lib_id "power:PWR_FLAG")
+		(at 129.54 48.26 0)
+		(unit 1)
+		(exclude_from_sim no)
+		(in_bom yes)
+		(on_board yes)
+		(dnp no)
+		(property "Reference" "#FLG074"
+			(at 129.54 46.355 0)
+			(effects
+				(font
+					(size 1.27 1.27)
+				)
+				(hide yes)
+			)
+		)
+		(property "Value" "PWR_FLAG"
+			(at 129.54 44.45 0)
+			(effects
+				(font
+					(size 1.27 1.27)
+				)
+				(hide yes)
+			)
+		)
+		(property "Footprint" ""
+			(at 129.54 48.26 0)
+			(effects
+				(font
+					(size 1.27 1.27)
+				)
+				(hide yes)
+			)
+		)
+		(property "Datasheet" "~"
+			(at 129.54 48.26 0)
+			(effects
+				(font
+					(size 1.27 1.27)
+				)
+				(hide yes)
+			)
+		)
+		(property "Description" "Special symbol for telling ERC where power comes from"
+			(at 129.54 48.26 0)
+			(effects
+				(font
+					(size 1.27 1.27)
+				)
+				(hide yes)
+			)
+		)
+		(pin "1"
+		)
+		(instances
+			(project "lincal"
+				(path "/b054cef4-39e3-49d8-aff0-7ba5a206c187/79d139b8-187a-44f5-bd99-1da7793824c6"
+					(reference "#FLG074")
+					(unit 1)
+				)
+			)
+		)
+	)
+	(symbol
 		(lib_id "Parts:+19V")
 		(at 240.03 43.18 0)
@@
 			)
 		)
-		(property "Value" "TestPoint"
+		(property "Value" "21V"
 			(at 134.62 38.1 0)
 			(effects
@@
 		(on_board yes)
 		(dnp no)
-		(property "Reference" "C523"
+		(property "Reference" "C54"
 			(at 170.18 49.022 0)
 			(effects
@@
 			(project "lincal"
 				(path "/b054cef4-39e3-49d8-aff0-7ba5a206c187/79d139b8-187a-44f5-bd99-1da7793824c6"
-					(reference "C523")
+					(reference "C54")
 					(unit 1)
 				)
@@
 	)
 	(symbol
+		(lib_id "power:PWR_FLAG")
+		(at 128.27 86.36 180)
+		(unit 1)
+		(exclude_from_sim no)
+		(in_bom yes)
+		(on_board yes)
+		(dnp no)
+		(property "Reference" "#FLG075"
+			(at 128.27 88.265 0)
+			(effects
+				(font
+					(size 1.27 1.27)
+				)
+				(hide yes)
+			)
+		)
+		(property "Value" "PWR_FLAG"
+			(at 128.27 90.17 0)
+			(effects
+				(font
+					(size 1.27 1.27)
+				)
+				(hide yes)
+			)
+		)
+		(property "Footprint" ""
+			(at 128.27 86.36 0)
+			(effects
+				(font
+					(size 1.27 1.27)
+				)
+				(hide yes)
+			)
+		)
+		(property "Datasheet" "~"
+			(at 128.27 86.36 0)
+			(effects
+				(font
+					(size 1.27 1.27)
+				)
+				(hide yes)
+			)
+		)
+		(property "Description" "Special symbol for telling ERC where power comes from"
+			(at 128.27 86.36 0)
+			(effects
+				(font
+					(size 1.27 1.27)
+				)
+				(hide yes)
+			)
+		)
+		(pin "1"
+		)
+		(instances
+			(project "lincal"
+				(path "/b054cef4-39e3-49d8-aff0-7ba5a206c187/79d139b8-187a-44f5-bd99-1da7793824c6"
+					(reference "#FLG075")
+					(unit 1)
+				)
+			)
+		)
+	)
+	(symbol
 		(lib_id "Device:R")
 		(at 201.93 106.68 0)
@@
 			)
 		)
-		(property "Footprint" "Package_DFN_QFN:Texas_RGW0020A_VQFN-20-1EP_5x5mm_P0.65mm_EP3.15x3.15mm"
+		(property "Footprint" "Parts:Texas_RGW0020A_VQFN-20-1EP_5x5mm_P0.65mm_EP3.15x3.15mm"
 			(at 192.405 36.83 0)
 			(effects
@@
 			)
 		)
-		(property "Footprint" "Package_DFN_QFN:Texas_RGW0020A_VQFN-20-1EP_5x5mm_P0.65mm_EP3.15x3.15mm"
+		(property "Footprint" "Parts:Texas_RGW0020A_VQFN-20-1EP_5x5mm_P0.65mm_EP3.15x3.15mm"
 			(at 189.23 86.36 0)
 			(effects

Commit message: More component metadata.
Parts:
- C50, C502, C503, C505, C508, C51, C511, C512, C52, C522, C524, C525, C526, C527, C528, C529, C53, C530, C54, C541, C542, C543, C544, C545, C546, C547, C548, C549, C550, C551, D53, D54, D56, D57, L53, L54, L55, L56, L57, L58, R503, R505, R511, R514, R542, U51, U52, U53: Stock (none) -> JLC
- R501: LCSC (none) -> C23147; Stock (none) -> JLC
- R502, R512: LCSC (none) -> C23172; Stock (none) -> JLC
- R541: LCSC (none) -> C25808; Stock (none) -> JLC
- R543: LCSC (none) -> C25811; Stock (none) -> JLC
- TP51, TP52, TP53, TP54: Stock - -> Board
Changed lines of the file:
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@@
 			)
 		)
-		(property "Stock" ""
+		(property "Stock" "JLC"
 			(at 154.94 43.18 90)
 			(effects
@@
 			)
 		)
-		(property "Stock" "-"
+		(property "Stock" "Board"
 			(at 134.62 92.71 0)
 			(effects
@@
 			)
 		)
-		(property "LCSC" ""
+		(property "LCSC" "C23172"
 			(at 118.11 59.69 90)
 			(effects
@@
 			)
 		)
-		(property "Stock" ""
+		(property "Stock" "JLC"
 			(at 118.11 59.69 90)
 			(effects
@@
 			)
 		)
-		(property "Stock" ""
+		(property "Stock" "JLC"
 			(at 123.19 52.07 90)
 			(effects
@@
 			)
 		)
-		(property "Stock" ""
+		(property "Stock" "JLC"
 			(at 64.77 78.74 90)
 			(effects
@@
 			)
 		)
-		(property "LCSC" ""
+		(property "LCSC" "C23172"
 			(at 118.11 74.93 90)
 			(effects
@@
 			)
 		)
-		(property "Stock" ""
+		(property "Stock" "JLC"
 			(at 118.11 74.93 90)
 			(effects
@@
 			)
 		)
-		(property "Stock" ""
+		(property "Stock" "JLC"
 			(at 134.62 55.88 0)
 			(effects
@@
 			)
 		)
-		(property "Stock" ""
+		(property "Stock" "JLC"
 			(at 154.94 96.52 0)
 			(effects
@@
 			)
 		)
-		(property "Stock" ""
+		(property "Stock" "JLC"
 			(at 96.52 63.5 0)
 			(effects
@@
 			)
 		)
-		(property "Stock" ""
+		(property "Stock" "JLC"
 			(at 129.54 55.88 0)
 			(effects
@@
 			)
 		)
-		(property "Stock" ""
+		(property "Stock" "JLC"
 			(at 201.93 114.3 90)
 			(effects
@@
 			)
 		)
-		(property "Stock" "-"
+		(property "Stock" "Board"
 			(at 223.52 92.71 0)
 			(effects
@@
 			)
 		)
-		(property "Stock" ""
+		(property "Stock" "JLC"
 			(at 228.6 96.52 0)
 			(effects
@@
 			)
 		)
-		(property "Stock" ""
+		(property "Stock" "JLC"
 			(at 146.05 86.36 90)
 			(effects
@@
 			)
 		)
-		(property "Stock" ""
+		(property "Stock" "JLC"
 			(at 64.77 60.96 90)
 			(effects
@@
 			)
 		)
-		(property "Stock" "-"
+		(property "Stock" "Board"
 			(at 223.52 43.18 0)
 			(effects
@@
 			)
 		)
-		(property "Stock" ""
+		(property "Stock" "JLC"
 			(at 233.68 46.99 0)
 			(effects
@@
 			)
 		)
-		(property "Stock" ""
+		(property "Stock" "JLC"
 			(at 160.02 92.71 90)
 			(effects
@@
 			)
 		)
-		(property "Stock" ""
+		(property "Stock" "JLC"
 			(at 123.19 82.55 90)
 			(effects
@@
 			)
 		)
-		(property "Stock" ""
+		(property "Stock" "JLC"
 			(at 228.6 46.99 0)
 			(effects
@@
 			)
 		)
-		(property "Stock" ""
+		(property "Stock" "JLC"
 			(at 139.7 74.93 0)
 			(effects
@@
 			)
 		)
-		(property "Stock" ""
+		(property "Stock" "JLC"
 			(at 171.45 96.52 0)
 			(effects
@@
 			)
 		)
-		(property "Stock" ""
+		(property "Stock" "JLC"
 			(at 149.86 92.71 90)
 			(effects
@@
 			)
 		)
-		(property "Stock" ""
+		(property "Stock" "JLC"
 			(at 64.77 43.18 90)
 			(effects
@@
 			)
 		)
-		(property "Stock" ""
+		(property "Stock" "JLC"
 			(at 177.8 109.22 0)
 			(effects
@@
 			)
 		)
-		(property "Stock" ""
+		(property "Stock" "JLC"
 			(at 218.44 46.99 0)
 			(effects
@@
 			)
 		)
-		(property "Stock" ""
+		(property "Stock" "JLC"
 			(at 128.27 74.93 0)
 			(effects
@@
 			)
 		)
-		(property "Stock" ""
+		(property "Stock" "JLC"
 			(at 165.1 96.52 0)
 			(effects
@@
 			)
 		)
-		(property "LCSC" ""
+		(property "LCSC" "C23147"
 			(at 73.66 43.18 90)
 			(effects
@@
 			)
 		)
-		(property "Stock" ""
+		(property "Stock" "JLC"
 			(at 73.66 43.18 90)
 			(effects
@@
 			)
 		)
-		(property "Stock" ""
+		(property "Stock" "JLC"
 			(at 140.97 92.71 0)
 			(effects
@@
 			)
 		)
-		(property "Stock" ""
+		(property "Stock" "JLC"
 			(at 73.66 78.74 90)
 			(effects
@@
 			)
 		)
-		(property "Stock" ""
+		(property "Stock" "JLC"
 			(at 207.01 46.99 0)
 			(effects
@@
 			)
 		)
-		(property "Stock" ""
+		(property "Stock" "JLC"
 			(at 213.36 46.99 0)
 			(effects
@@
 			)
 		)
-		(property "Stock" ""
+		(property "Stock" "JLC"
 			(at 213.36 96.52 0)
 			(effects
@@
 			)
 		)
-		(property "Stock" "-"
+		(property "Stock" "Board"
 			(at 134.62 43.18 0)
 			(effects
@@
 			)
 		)
-		(property "Stock" ""
+		(property "Stock" "JLC"
 			(at 233.68 96.52 0)
 			(effects
@@
 			)
 		)
-		(property "Stock" ""
+		(property "Stock" "JLC"
 			(at 165.1 46.99 0)
 			(effects
@@
 			)
 		)
-		(property "Stock" ""
+		(property "Stock" "JLC"
 			(at 170.18 46.99 0)
 			(effects
@@
 			)
 		)
-		(property "Stock" ""
+		(property "Stock" "JLC"
 			(at 223.52 46.99 0)
 			(effects
@@
 			)
 		)
-		(property "Stock" ""
+		(property "Stock" "JLC"
 			(at 223.52 96.52 0)
 			(effects
@@
 			)
 		)
-		(property "Stock" ""
+		(property "Stock" "JLC"
 			(at 134.62 74.93 0)
 			(effects
@@
 			)
 		)
-		(property "Stock" ""
+		(property "Stock" "JLC"
 			(at 74.93 54.61 90)
 			(effects
@@
 			)
 		)
-		(property "Stock" ""
+		(property "Stock" "JLC"
 			(at 240.03 46.99 0)
 			(effects
@@
 			)
 		)
-		(property "Stock" ""
+		(property "Stock" "JLC"
 			(at 240.03 87.63 0)
 			(effects
@@
 			)
 		)
-		(property "Stock" ""
+		(property "Stock" "JLC"
 			(at 200.66 72.39 0)
 			(effects
@@
 			)
 		)
-		(property "Stock" ""
+		(property "Stock" "JLC"
 			(at 73.66 38.1 90)
 			(effects
@@
 			)
 		)
-		(property "Stock" ""
+		(property "Stock" "JLC"
 			(at 71.12 64.77 0)
 			(effects
@@
 			)
 		)
-		(property "Stock" ""
+		(property "Stock" "JLC"
 			(at 77.47 64.77 0)
 			(effects
@@
 			)
 		)
-		(property "Stock" ""
+		(property "Stock" "JLC"
 			(at 207.01 106.68 0)
 			(effects
@@
 			)
 		)
-		(property "LCSC" ""
+		(property "LCSC" "C25808"
 			(at 201.93 106.68 90)
 			(effects
@@
 			)
 		)
-		(property "Stock" ""
+		(property "Stock" "JLC"
 			(at 201.93 106.68 90)
 			(effects
@@
 			)
 		)
-		(property "Stock" ""
+		(property "Stock" "JLC"
 			(at 139.7 48.26 90)
 			(effects
@@
 			)
 		)
-		(property "Stock" ""
+		(property "Stock" "JLC"
 			(at 207.01 96.52 0)
 			(effects
@@
 			)
 		)
-		(property "Stock" ""
+		(property "Stock" "JLC"
 			(at 187.96 58.42 0)
 			(effects
@@
 			)
 		)
-		(property "Stock" ""
+		(property "Stock" "JLC"
 			(at 187.96 97.79 0)
 			(effects
@@
 			)
 		)
-		(property "LCSC" ""
+		(property "LCSC" "C25811"
 			(at 207.01 114.3 90)
 			(effects
@@
 			)
 		)
-		(property "Stock" ""
+		(property "Stock" "JLC"
 			(at 207.01 114.3 90)
 			(effects
@@
 			)
 		)
-		(property "Stock" ""
+		(property "Stock" "JLC"
 			(at 218.44 96.52 0)
 			(effects
@@
 			)
 		)
-		(property "Stock" ""
+		(property "Stock" "JLC"
 			(at 140.97 43.18 0)
 			(effects

Commit message: Front panel
Parts:
- renumbered TP54 to -16V1, TP53 to -18V1, TP52 to 19V1, TP51 to 21V1
Other:
- moved on the sheet: L58
Changed lines of the file:
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@@
 	(wire
 		(pts
-			(xy 149.86 86.36) (xy 151.13 86.36)
+			(xy 148.59 86.36) (xy 149.86 86.36)
 		)
 		(stroke
@@
 	(wire
 		(pts
-			(xy 142.24 86.36) (xy 139.7 86.36)
+			(xy 140.97 86.36) (xy 139.7 86.36)
 		)
 		(stroke
@@
 	(global_label "-18V"
 		(shape output)
-		(at 151.13 86.36 0)
+		(at 149.86 86.36 0)
 		(effects
 			(font
@@
 		)
 		(property "Intersheetrefs" "${INTERSHEET_REFS}"
-			(at 158.6872 86.36 0)
+			(at 157.4172 86.36 0)
 			(effects
 				(font
@@
 		(on_board yes)
 		(dnp no)
-		(property "Reference" "TP53"
+		(property "Reference" "-18V1"
 			(at 134.62 98.044 0)
 			(effects
@@
 					(size 1.27 1.27)
 				)
+				(hide yes)
 			)
 		)
@@
 					(size 1.27 1.27)
 				)
-				(hide yes)
 			)
 		)
@@
 			(project "lincal"
 				(path "/b054cef4-39e3-49d8-aff0-7ba5a206c187/79d139b8-187a-44f5-bd99-1da7793824c6"
-					(reference "TP53")
+					(reference "-18V1")
 					(unit 1)
 				)
@@
 		(on_board yes)
 		(dnp no)
-		(property "Reference" "TP54"
+		(property "Reference" "-16V1"
 			(at 223.52 87.376 0)
 			(effects
@@
 					(size 1.27 1.27)
 				)
+				(hide yes)
 			)
 		)
@@
 					(size 1.27 1.27)
 				)
-				(hide yes)
 			)
 		)
@@
 			(project "lincal"
 				(path "/b054cef4-39e3-49d8-aff0-7ba5a206c187/79d139b8-187a-44f5-bd99-1da7793824c6"
-					(reference "TP54")
+					(reference "-16V1")
 					(unit 1)
 				)
@@
 	(symbol
 		(lib_id "Parts:L_Ferrite_Power")
-		(at 146.05 86.36 90)
+		(at 144.78 86.36 90)
 		(unit 1)
 		(exclude_from_sim no)
@@
 		(dnp no)
 		(property "Reference" "L58"
-			(at 146.05 87.63 90)
+			(at 144.78 87.63 90)
 			(effects
 				(font
@@
 		)
 		(property "Value" "100"
-			(at 146.05 83.566 90)
+			(at 144.78 83.566 90)
 			(effects
 				(font
@@
 		)
 		(property "Footprint" "Inductor_SMD:L_0603_1608Metric"
-			(at 146.05 86.36 0)
+			(at 144.78 86.36 0)
 			(effects
 				(font
@@
 		)
 		(property "Datasheet" "2A / 50mΩ"
-			(at 146.05 86.36 0)
+			(at 144.78 86.36 0)
 			(effects
 				(font
@@
 		)
 		(property "Description" "Inductor with ferrite core"
-			(at 146.05 86.36 0)
+			(at 144.78 86.36 0)
 			(effects
 				(font
@@
 		)
 		(property "LCSC" "C14709"
-			(at 146.05 86.36 90)
+			(at 144.78 86.36 90)
 			(effects
 				(font
@@
 		)
 		(property "Stock" "JLC"
-			(at 146.05 86.36 90)
+			(at 144.78 86.36 90)
 			(effects
 				(font
@@
 		(on_board yes)
 		(dnp no)
-		(property "Reference" "TP52"
+		(property "Reference" "19V1"
 			(at 223.52 37.592 0)
 			(effects
@@
 					(size 1.27 1.27)
 				)
+				(hide yes)
 			)
 		)
@@
 					(size 1.27 1.27)
 				)
-				(hide yes)
 			)
 		)
@@
 			(project "lincal"
 				(path "/b054cef4-39e3-49d8-aff0-7ba5a206c187/79d139b8-187a-44f5-bd99-1da7793824c6"
-					(reference "TP52")
+					(reference "19V1")
 					(unit 1)
 				)
@@
 		(on_board yes)
 		(dnp no)
-		(property "Reference" "TP51"
+		(property "Reference" "21V1"
 			(at 134.62 37.846 0)
 			(effects
@@
 					(size 1.27 1.27)
 				)
+				(hide yes)
 			)
 		)
@@
 					(size 1.27 1.27)
 				)
-				(hide yes)
 			)
 		)
@@
 			(project "lincal"
 				(path "/b054cef4-39e3-49d8-aff0-7ba5a206c187/79d139b8-187a-44f5-bd99-1da7793824c6"
-					(reference "TP51")
+					(reference "21V1")
 					(unit 1)
 				)

Commit message: Tweak various feedback loops.
Parts:
- U52, U53: now in the parts list
Changed lines of the file:
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@@
 		(unit 1)
 		(exclude_from_sim no)
-		(in_bom no)
+		(in_bom yes)
 		(on_board yes)
 		(dnp no)
@@
 		(unit 1)
 		(exclude_from_sim no)
-		(in_bom no)
+		(in_bom yes)
 		(on_board yes)
 		(dnp no)

Commit message: Readyish
Parts:
- C545: LCSC C307500 -> C389113
- U52: LCSC C114839 -> C28286
Changed lines of the file:
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@@
 			)
 		)
-		(property "Datasheet" "C0G, 25V"
+		(property "Datasheet" "C0G, 50V"
 			(at 207.01 106.68 0)
 			(effects
@@
 			)
 		)
-		(property "LCSC" "C307500"
+		(property "LCSC" "C389113"
 			(at 207.01 106.68 0)
 			(effects
@@
 			)
 		)
-		(property "LCSC" "C114839"
+		(property "LCSC" "C28286"
 			(at 187.96 58.42 0)
 			(effects
