File: end-digi.kicad_pcb (KiCad board)
At the start: 2 copper layers, 160 x 80 mm, 7 parts

Commit message: Contact pads.  Shuffle the big cap.
Other:
- board text added: "Cal"
- board text added: "Lin"
Changed lines of the file:
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@@
+			(thermal_bridge_angle 90)
+		)
+		(pad "1" smd circle
+			(at 0 0)
+			(size 10 10)
+			(layers "F.Cu" "F.Mask")
+			(net 2 "Earth")
+			(pinfunction "1")
+			(pintype "input")
 			(thermal_bridge_angle 90)
 		)
@@
 			(thermal_bridge_angle 90)
 		)
+		(pad "1" smd circle
+			(at 0 0)
+			(size 10 10)
+			(layers "F.Cu" "F.Mask")
+			(net 2 "Earth")
+			(pinfunction "1")
+			(pintype "input")
+			(thermal_bridge_angle 90)
+		)
 		(embedded_fonts no)
 	)
@@
 			(pinfunction "1")
 			(pintype "input")
-			(solder_mask_margin 0)
 			(clearance 1.4)
+			(thermal_bridge_angle 90)
+		)
+		(pad "1" smd circle
+			(at 0 0)
+			(size 10 10)
+			(layers "F.Cu" "F.Mask")
+			(net 1 "GNDPWR")
+			(pinfunction "1")
+			(pintype "input")
 			(thermal_bridge_angle 90)
 		)
@@
 		(embedded_fonts no)
 	)
-	(gr_circle
-		(center 85 67.45)
-		(end 90 67.45)
+	(gr_rect
+		(start 167 72)
+		(end 171 74)
 		(stroke
 			(width 0)
@@
 		)
 		(fill yes)
-		(layers "F.Cu" "F.Mask")
-		(net 2)
-	)
-	(gr_circle
-		(center 115 67.45)
-		(end 120 67.45)
-		(stroke
-			(width 0)
-			(type default)
-		)
-		(fill yes)
-		(layers "F.Cu" "F.Mask")
-		(net 1)
-	)
-	(gr_circle
-		(center 100 67.45)
-		(end 105 67.45)
-		(stroke
-			(width 0)
-			(type default)
-		)
-		(fill yes)
-		(layers "F.Cu" "F.Mask")
-		(net 2)
+		(layer "B.Mask")
 	)
 	(gr_line
@@
 		(locked yes)
 		(layer "User.1")
+	)
+	(gr_text "Lin"
+		(at 206 67.45 0)
+		(layer "F.SilkS")
+		(effects
+			(font
+				(size 5 5)
+				(thickness 1)
+				(bold yes)
+			)
+			(justify right)
+		)
 	)
 	(gr_text "Ant."
@@
 			)
 			(justify left bottom)
+		)
+	)
+	(gr_text "Cal"
+		(at 205 67.45 0)
+		(layer "F.SilkS")
+		(effects
+			(font
+				(size 5 5)
+				(thickness 1)
+				(bold yes)
+				(italic yes)
+			)
+			(justify left)
 		)
 	)
@@
 	(dimension
 		(type orthogonal)
-		(locked yes)
 		(layer "User.1")
 		(pts
 			(xy 72.2 69.6) (xy 72.2 62)
 		)
-		(height -14.95)
+		(height -9.2)
 		(orientation 1)
 		(format
@@
 		)
 		(gr_text "7.6"
-			(locked yes)
-			(at 56.1 65.8 90)
+			(at 61.85 65.8 90)
 			(layer "User.1")
 			(effects
@@
 			(xy 230 60) (xy 230 140)
 		)
-		(height 38.05)
+		(height 13)
 		(orientation 1)
 		(format
@@
 		(gr_text "80"
 			(locked yes)
-			(at 266.9 100 90)
+			(at 241.85 100 90)
 			(layer "User.1")
 			(effects
@@
 			(xy 225.3 64.5) (xy 225.3 135.5)
 		)
-		(height 33.9)
+		(height 13.7)
 		(orientation 1)
 		(format
@@
 		(gr_text "71"
 			(locked yes)
-			(at 258.05 100 90)
+			(at 237.85 100 90)
 			(layer "User.1")
 			(effects
@@
 	(dimension
 		(type orthogonal)
-		(locked yes)
 		(layer "User.1")
 		(pts
 			(xy 72.2 138) (xy 72.2 130.4)
 		)
-		(height -14.95)
+		(height -9.2)
 		(orientation 1)
 		(format
@@
 		)
 		(gr_text "7.6"
-			(locked yes)
-			(at 56.1 134.2 90)
+			(at 61.85 134.2 90)
 			(layer "User.1")
 			(effects
@@
 		(min_thickness 0.25)
 		(filled_areas_thickness no)
-		(fill yes
+		(fill
 			(thermal_gap 0.5)
 			(thermal_bridge_width 0.5)
@@
 		(polygon
 			(pts
-				(xy 65 55) (xy 235 55) (xy 235 170) (xy 65 170)
-			)
-		)
+				(xy 65 55) (xy 235 55) (xy 235 145) (xy 65 145)
+			)
+		)
